File: eagle/joesTriac-2nd/powerBoard-2nd.sch (EAGLE design)
At the start: 6 parts, among them J1 XF2E-0815-1

Commit message: reg save
Parts:
- added IC1: 7809, v-reg:78LXX
- added IC2: 7805, v-reg:78LXX
- added IC3: 7909, v-reg:79LXX
- added IC4: (no value), v-reg:LM317-T039
- added IC6: (no value), v-reg:LM337-TO3
- added J2: XF2E-0815-1, con-omron:XF2E-0815-1
- added R1, R2, R3, R4: (no value), resistor:R-EU_0309/V
Connections:
- new net +9V: IC1.OUT, IC4.IN, J2-7.MS
- new net -9V: IC3.OUT, IC6.IN, J2-6.MS
- new net N$10: IC2.OUT, J2-4.MS
- new net N$18: IC4.ADJ, R1.1, R2.2
- new net N$19: IC6.ADJ, R3.1, R4.2
- new net N$21: IC6.OUT, J2-3.MS
- new net N$23: IC4.OUT, J2-8.MS
- net +12V: now also IC1.IN, IC2.IN
- net -12V: now also IC3.IN
- net GND: now also IC1.GND, IC2.GND, IC3.GND, J2-5.MS, R2.1, R3.2
Other:
- note added: "+2.5V"
- note added: "-2.5V"
- moved on the sheet: B1, F1, F2, F3, J1-1, J1-2, J1-3, J1-4, J1-5, J1-6, J1-7, J1-8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

Commit message: reg save
Parts:
- added M1: (no value), e-motoren:MOTOR_1-PHASEN
Connections:
- net GND: now also M1.V
- net N$10: now also M1.U
Other:
- note added: "Ventilator"
Changed lines of the file:
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@@
 <part name="R3" library="resistor" deviceset="R-EU_" device="0309/V"/>
 <part name="R4" library="resistor" deviceset="R-EU_" device="0309/V"/>
+<part name="M1" library="e-motoren" deviceset="MOTOR_1-PHASEN" device=""/>
+<part name="SUPPLY12" library="supply2" deviceset="GND" device=""/>
 </parts>
 <sheets>
@@
 <text x="10.16" y="-5.08" size="1.778" layer="91">  +2.5V</text>
 <text x="5.08" y="-48.26" size="1.778" layer="91">  -2.5V</text>
+<text x="71.12" y="-38.1" size="2.54" layer="91">Ventilator</text>
 </plain>
 <instances>
@@
 <instance part="R3" gate="G$1" x="-7.62" y="-33.02" rot="R90"/>
 <instance part="R4" gate="G$1" x="5.08" y="-40.64" rot="R90"/>
+<instance part="M1" gate="1" x="68.58" y="-25.4"/>
+<instance part="SUPPLY12" gate="GND" x="88.9" y="-25.4"/>
 </instances>
 <busses>
@@
 <wire x1="-73.66" y1="-12.7" x2="-88.9" y2="-12.7" width="0.1524" layer="91"/>
 </segment>
+<segment>
+<pinref part="M1" gate="1" pin="V"/>
+<wire x1="71.12" y1="-17.78" x2="71.12" y2="-12.7" width="0.1524" layer="91"/>
+<wire x1="71.12" y1="-12.7" x2="88.9" y2="-12.7" width="0.1524" layer="91"/>
+<wire x1="88.9" y1="-12.7" x2="88.9" y2="-22.86" width="0.1524" layer="91"/>
+<pinref part="SUPPLY12" gate="GND" pin="GND"/>
+</segment>
 </net>
 <net name="+12V" class="0">
@@
 <pinref part="J2" gate="-4" pin="MS"/>
 <wire x1="-76.2" y1="-15.24" x2="-88.9" y2="-15.24" width="0.1524" layer="91"/>
+<wire x1="50.8" y1="-7.62" x2="66.04" y2="-7.62" width="0.1524" layer="91"/>
+<pinref part="M1" gate="1" pin="U"/>
+<wire x1="66.04" y1="-7.62" x2="66.04" y2="-17.78" width="0.1524" layer="91"/>
 </segment>
 </net>
@@
 <pinref part="IC4" gate="G$1" pin="OUT"/>
 <wire x1="5.08" y1="-7.62" x2="7.62" y2="-7.62" width="0.1524" layer="91"/>
-<wire x1="7.62" y1="-7.62" x2="12.7" y2="-7.62" width="0.1524" layer="91"/>
+<wire x1="7.62" y1="-7.62" x2="10.16" y2="-7.62" width="0.1524" layer="91"/>
 <wire x1="7.62" y1="-7.62" x2="7.62" y2="2.54" width="0.1524" layer="91"/>
 <wire x1="7.62" y1="2.54" x2="-17.78" y2="2.54" width="0.1524" layer="91"/>

Commit message: reg save
Parts:
- added C1, C2, C5: 1100uF, resistor:CPOL-EUE22-6AXIAL
- added C11, C3, C6, C8, C9: (no value), resistor:CPOL-EUE22-6AXIAL
Connections:
- removed net N$10: IC2.OUT, J2-4.MS, M1.U
- new net +5V: C5.+, IC2.OUT, J2-4.MS
- net +12V: now also C3.+, C9.+, M1.U
- net +9V: now also C1.+
- net -12V: now also C11.-
- net -9V: now also C2.-
- net GND: now also C1.-, C2.+, C3.-, C5.-, C6.-, C8.+, C9.-
- net N$21: now also C8.-, R4.1
- net N$23: now also C6.+
Other:
- moved on the sheet: M1

Commit message: reg save
Parts:
- added C10, C4, C7: (no value), resistor:CPOL-EUE22-6AXIAL
- added IC5: 7809, v-reg:78LXX
- added R5: (no value), resistor:R-EU_0309/V
- added R9: (no value), resistor:R-TRIMM4G/J
Connections:
- new net N$16: C7.+, IC5.OUT, M1.V, R5.2
- new net N$17: IC5.GND, R5.1, R9.E
- net +12V: now also C4.+; no longer M1.U
- net -12V: now also C10.-, C7.-, M1.U, R9.S
- net GND: now also C10.+, IC5.IN; no longer M1.V
Other:
- note added: "/+16V"
- note added: "/-16V"
- moved on the sheet: M1
Changed lines of the file:
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@@
 <layer number="97" name="Info" color="7" fill="1" visible="yes" active="yes"/>
 <layer number="98" name="Guide" color="6" fill="1" visible="yes" active="yes"/>
+<layer number="99" name="SpiceOrder" color="5" fill="1" visible="yes" active="yes"/>
 </layers>
 <schematic xreflabel="%F%N/%S.%C%R" xrefpart="/%S.%C%R">
@@
 <part name="SUPPLY1" library="supply2" deviceset="GND" device=""/>
 <part name="SUPPLY2" library="supply2" deviceset="GND" device=""/>
-<part name="SUPPLY4" library="supply2" deviceset="+12V" device=""/>
-<part name="SUPPLY3" library="supply2" deviceset="-12V" device=""/>
-<part name="SUPPLY5" library="supply2" deviceset="-12V" device=""/>
+<part name="SUPPLY4" library="supply2" deviceset="+12V" device="" value="+16V"/>
 <part name="SUPPLY6" library="supply2" deviceset="+12V" device=""/>
 <part name="SUPPLY7" library="supply2" deviceset="-12V" device=""/>
@@
 <part name="R4" library="resistor" deviceset="R-EU_" device="0309/V"/>
 <part name="M1" library="e-motoren" deviceset="MOTOR_1-PHASEN" device=""/>
-<part name="SUPPLY12" library="supply2" deviceset="GND" device=""/>
 <part name="C1" library="resistor" deviceset="CPOL-EU" device="E22-6AXIAL" value="1100uF"/>
 <part name="C2" library="resistor" deviceset="CPOL-EU" device="E22-6AXIAL" value="1100uF"/>
@@
 <part name="SUPPLY13" library="supply2" deviceset="+5V" device=""/>
 <part name="C5" library="resistor" deviceset="CPOL-EU" device="E22-6AXIAL" value="1100uF"/>
+<part name="IC5" library="v-reg" deviceset="78LXX" device="" value="7809"/>
+<part name="SUPPLY14" library="supply2" deviceset="GND" device=""/>
+<part name="SUPPLY15" library="supply2" deviceset="-12V" device="" value="-16V"/>
+<part name="R5" library="resistor" deviceset="R-EU_" device="0309/V"/>
+<part name="R9" library="resistor" deviceset="R-TRIMM" device="4G/J"/>
+<part name="C4" library="resistor" deviceset="CPOL-EU" device="E22-6AXIAL"/>
+<part name="SUPPLY12" library="supply2" deviceset="GND" device=""/>
+<part name="C10" library="resistor" deviceset="CPOL-EU" device="E22-6AXIAL"/>
+<part name="SUPPLY16" library="supply2" deviceset="GND" device=""/>
+<part name="SUPPLY3" library="supply2" deviceset="-12V" device="" value="-16V"/>
+<part name="C7" library="resistor" deviceset="CPOL-EU" device="E22-6AXIAL"/>
 </parts>
 <sheets>
@@
 <text x="-53.34" y="38.1" size="1.778" layer="91">220V 50Hz AC</text>
 <text x="10.16" y="-5.08" size="1.778" layer="91">  +2.5V</text>
-<text x="76.2" y="-38.1" size="2.54" layer="91">Ventilator</text>
+<text x="81.28" y="-48.26" size="2.54" layer="91">Ventilator</text>
 <text x="5.08" y="-50.8" size="1.778" layer="91">  -2.5V</text>
+<text x="-50.8" y="-2.54" size="1.778" layer="91">/+16V</text>
+<text x="-53.34" y="-53.34" size="1.778" layer="91">/-16V</text>
 </plain>
 <instances>
@@
 <instance part="SUPPLY2" gate="GND" x="43.18" y="22.86"/>
 <instance part="SUPPLY4" gate="+12V" x="15.24" y="20.32"/>
-<instance part="SUPPLY3" gate="G$1" x="-2.54" y="17.78"/>
-<instance part="SUPPLY5" gate="G$1" x="-2.54" y="17.78"/>
 <instance part="SUPPLY6" gate="+12V" x="-55.88" y="-5.08"/>
 <instance part="SUPPLY7" gate="G$1" x="-55.88" y="-48.26"/>
@@
 <instance part="R3" gate="G$1" x="-7.62" y="-33.02" rot="R90"/>
 <instance part="R4" gate="G$1" x="5.08" y="-40.64" rot="R90"/>
-<instance part="M1" gate="1" x="73.66" y="-25.4"/>
-<instance part="SUPPLY12" gate="GND" x="93.98" y="-25.4"/>
+<instance part="M1" gate="1" x="116.84" y="-7.62"/>
 <instance part="C1" gate="G$1" x="-30.48" y="-15.24"/>
 <instance part="C2" gate="G$1" x="-30.48" y="-35.56"/>
@@
 <instance part="SUPPLY13" gate="+5V" x="50.8" y="-5.08"/>
 <instance part="C5" gate="G$1" x="53.34" y="-15.24"/>
+<instance part="IC5" gate="1" x="86.36" y="10.16"/>
+<instance part="SUPPLY14" gate="GND" x="76.2" y="7.62"/>
+<instance part="SUPPLY15" gate="G$1" x="99.06" y="-25.4"/>
+<instance part="R5" gate="G$1" x="99.06" y="5.08" rot="R90"/>
+<instance part="R9" gate="G$1" x="86.36" y="-5.08"/>
+<instance part="C4" gate="G$1" x="12.7" y="15.24"/>
+<instance part="SUPPLY12" gate="GND" x="12.7" y="10.16"/>
+<instance part="C10" gate="G$1" x="-12.7" y="15.24" rot="R180"/>
+<instance part="SUPPLY16" gate="GND" x="-12.7" y="10.16"/>
+<instance part="SUPPLY3" gate="G$1" x="-2.54" y="17.78"/>
+<instance part="C7" gate="G$1" x="104.14" y="-7.62"/>
 </instances>
 <busses>
@@
 <wire x1="40.64" y1="25.4" x2="40.64" y2="22.86" width="0.1524" layer="91"/>
 <wire x1="40.64" y1="25.4" x2="43.18" y2="25.4" width="0.1524" layer="91"/>
-</segment>
-<segment>
-<pinref part="M1" gate="1" pin="V"/>
-<wire x1="76.2" y1="-17.78" x2="76.2" y2="-12.7" width="0.1524" layer="91"/>
-<wire x1="76.2" y1="-12.7" x2="93.98" y2="-12.7" width="0.1524" layer="91"/>
-<wire x1="93.98" y1="-12.7" x2="93.98" y2="-22.86" width="0.1524" layer="91"/>
-<pinref part="SUPPLY12" gate="GND" pin="GND"/>
 </segment>
 <segment>
@@
 <wire x1="53.34" y1="-27.94" x2="53.34" y2="-20.32" width="0.1524" layer="91"/>
 </segment>
+<segment>
+<pinref part="SUPPLY14" gate="GND" pin="GND"/>
+<pinref part="IC5" gate="1" pin="IN"/>
+<wire x1="76.2" y1="10.16" x2="78.74" y2="10.16" width="0.1524" layer="91"/>
+</segment>
+<segment>
+<pinref part="C10" gate="G$1" pin="+"/>
+<pinref part="SUPPLY16" gate="GND" pin="GND"/>
+</segment>
 </net>
 <net name="+12V" class="0">
@@
 <wire x1="10.16" y1="25.4" x2="10.16" y2="17.78" width="0.1524" layer="91"/>
 <pinref part="SUPPLY4" gate="+12V" pin="+12V"/>
-<wire x1="10.16" y1="17.78" x2="15.24" y2="17.78" width="0.1524" layer="91"/>
+<wire x1="10.16" y1="17.78" x2="12.7" y2="17.78" width="0.1524" layer="91"/>
+<pinref part="C4" gate="G$1" pin="+"/>
+<wire x1="12.7" y1="17.78" x2="15.24" y2="17.78" width="0.1524" layer="91"/>
+<junction x="12.7" y="17.78"/>
 </segment>
 <segment>
@@
 </segment>
 <segment>
+<pinref part="SUPPLY9" gate="+12V" pin="+12V"/>
 <pinref part="IC2" gate="1" pin="IN"/>
 <wire x1="30.48" y1="-7.62" x2="27.94" y2="-7.62" width="0.1524" layer="91"/>
-<pinref part="SUPPLY9" gate="+12V" pin="+12V"/>
+<wire x1="27.94" y1="-7.62" x2="25.4" y2="-7.62" width="0.1524" layer="91"/>
 <pinref part="C3" gate="G$1" pin="+"/>
-<wire x1="27.94" y1="-7.62" x2="25.4" y2="-7.62" width="0.1524" layer="91"/>
 <wire x1="27.94" y1="-12.7" x2="27.94" y2="-7.62" width="0.1524" layer="91"/>
-<wire x1="30.48" y1="-7.62" x2="30.48" y2="2.54" width="0.1524" layer="91"/>
-<wire x1="30.48" y1="2.54" x2="71.12" y2="2.54" width="0.1524" layer="91"/>
-<pinref part="M1" gate="1" pin="U"/>
-<wire x1="71.12" y1="-7.62" x2="71.12" y2="-10.16" width="0.1524" layer="91"/>
-<wire x1="71.12" y1="-10.16" x2="71.12" y2="-17.78" width="0.1524" layer="91"/>
-<wire x1="71.12" y1="2.54" x2="71.12" y2="-7.62" width="0.1524" layer="91"/>
 </segment>
 </net>
 <net name="-12V" class="0">
-<segment>
-<pinref part="SUPPLY3" gate="G$1" pin="-12V"/>
-<pinref part="SUPPLY5" gate="G$1" pin="-12V"/>
-<pinref part="J1" gate="-3" pin="MS"/>
-<wire x1="-17.78" y1="20.32" x2="-2.54" y2="20.32" width="0.1524" layer="91"/>
-</segment>
 <segment>
 <pinref part="SUPPLY7" gate="G$1" pin="-12V"/>
@@
 <pinref part="C11" gate="G$1" pin="-"/>
 <wire x1="-55.88" y1="-43.18" x2="-55.88" y2="-45.72" width="0.1524" layer="91"/>
+</segment>
+<segment>
+<wire x1="81.28" y1="-22.86" x2="91.44" y2="-22.86" width="0.1524" layer="91"/>
+<wire x1="91.44" y1="-22.86" x2="99.06" y2="-22.86" width="0.1524" layer="91"/>
+<pinref part="SUPPLY15" gate="G$1" pin="-12V"/>
+<pinref part="R9" gate="G$1" pin="S"/>
+<wire x1="91.44" y1="-5.08" x2="91.44" y2="-22.86" width="0.1524" layer="91"/>
+<pinref part="C7" gate="G$1" pin="-"/>
+<wire x1="104.14" y1="-12.7" x2="104.14" y2="-22.86" width="0.1524" layer="91"/>
+<wire x1="104.14" y1="-22.86" x2="99.06" y2="-22.86" width="0.1524" layer="91"/>
+<pinref part="M1" gate="1" pin="U"/>
+<wire x1="114.3" y1="0" x2="109.22" y2="0" width="0.1524" layer="91"/>
+<wire x1="109.22" y1="0" x2="109.22" y2="-22.86" width="0.1524" layer="91"/>
+<wire x1="109.22" y1="-22.86" x2="104.14" y2="-22.86" width="0.1524" layer="91"/>
+</segment>
+<segment>
+<pinref part="J1" gate="-3" pin="MS"/>
+<wire x1="-17.78" y1="20.32" x2="-12.7" y2="20.32" width="0.1524" layer="91"/>
+<pinref part="C10" gate="G$1" pin="-"/>
+<wire x1="-12.7" y1="20.32" x2="-2.54" y2="20.32" width="0.1524" layer="91"/>
+<junction x="-12.7" y="20.32"/>
+<pinref part="SUPPLY3" gate="G$1" pin="-12V"/>
 </segment>
 </net>
@@
 </segment>
 </net>
+<net name="N$16" class="0">
+<segment>
+<pinref part="IC5" gate="1" pin="OUT"/>
+<pinref part="R5" gate="G$1" pin="2"/>
+<wire x1="93.98" y1="10.16" x2="99.06" y2="10.16" width="0.1524" layer="91"/>
+<wire x1="99.06" y1="10.16" x2="104.14" y2="10.16" width="0.1524" layer="91"/>
+<pinref part="C7" gate="G$1" pin="+"/>
+<wire x1="104.14" y1="10.16" x2="104.14" y2="-5.08" width="0.1524" layer="91"/>
+<wire x1="104.14" y1="10.16" x2="119.38" y2="10.16" width="0.1524" layer="91"/>
+<pinref part="M1" gate="1" pin="V"/>
+<wire x1="119.38" y1="10.16" x2="119.38" y2="0" width="0.1524" layer="91"/>
+</segment>
+</net>
+<net name="N$17" class="0">
+<segment>
+<pinref part="IC5" gate="1" pin="GND"/>
+<pinref part="R9" gate="G$1" pin="E"/>
+<wire x1="86.36" y1="2.54" x2="86.36" y2="0" width="0.1524" layer="91"/>
+<pinref part="R5" gate="G$1" pin="1"/>
+<wire x1="99.06" y1="0" x2="99.06" y2="-2.54" width="0.1524" layer="91"/>
+<wire x1="99.06" y1="-2.54" x2="88.9" y2="-2.54" width="0.1524" layer="91"/>
+<wire x1="88.9" y1="-2.54" x2="88.9" y2="0" width="0.1524" layer="91"/>
+<wire x1="88.9" y1="0" x2="86.36" y2="0" width="0.1524" layer="91"/>
+</segment>
+</net>
+<net name="N$24" class="0">
+<segment>
+<wire x1="76.2" y1="-7.62" x2="73.66" y2="-7.62" width="0.1524" layer="91"/>
+</segment>
+</net>

Commit message: reg save
Changed lines of the file:
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@@
 <text x="-53.34" y="38.1" size="1.778" layer="91">220V 50Hz AC</text>
 <text x="10.16" y="-5.08" size="1.778" layer="91">  +2.5V</text>
-<text x="81.28" y="-48.26" size="2.54" layer="91">Ventilator</text>
+<text x="111.76" y="-22.86" size="2.54" layer="91">Ventilator</text>
 <text x="5.08" y="-50.8" size="1.778" layer="91">  -2.5V</text>
 <text x="-50.8" y="-2.54" size="1.778" layer="91">/+16V</text>

Commit message: reg save
Parts:
- added R6, R7: (no value), resistor:R-TRIMM4G/J
Connections:
- new net N$10: R3.1, R7.E
- new net N$20: IC6.ADJ, R4.2, R7.S
- net GND: now also C11.+; no longer R2.1
- net N$18: now also R6.S; no longer R2.2
- net N$19: now also R2.2, R6.A; no longer IC6.ADJ, R3.1, R4.2
- net N$23: now also R1.2
Other:
- moved on the sheet: B1, C1, C10, C11, C2, C3, C4, C5, C6, C7, C8, C9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

Commit message: reg save
Parts:
- added D1, D2: 1N4446, diode:1N4446
- added D3: 1N4736_Zener_6.8V, diode:1N4446
- added IC7: LM311N, linear:LM311N
- added R10: (no value), resistor:R-TRIMM4G/J
- added R11, R13, R14, R15, R8: (no value), resistor:R-EU_0309/V
Connections:
- new net N$22: D3.C, IC7.-IN, R14.2, R15.1
- new net N$25: IC7.+IN, R10.S, R13.1
- new net N$26: R10.E, R8.1
- new net N$28: D1.C, D2.C, R15.2
- new net N$29: IC7.OUT, R11.1, R13.2
- net +5V: now also R11.2, R8.2
- net +9V: now also IC7.V+
- net -9V: now also IC7.V-
- net GND: now also D3.A, IC7.GND, R10.A, R14.1
- net N$3: now also D1.A
- net N$4: now also D2.A
Other:
- note added: "hysterese"
- note added: "zero pass signal"
- moved on the sheet: C7, IC5, M1, R5, R9

Commit message: reg save
Parts:
- added R16: 10k, resistor:R-EU_0309/V
- R10: value (none) -> 2k
- R11: value (none) -> 24k
- R13: value (none) -> 330k
- R14: value (none) -> 33k
- R15: value (none) -> 2.2k
- R8: value (none) -> 3.3k
Connections:
- new net N$27: R10.S, R16.2
- net N$25: now also R16.1; no longer R10.S
Other:
- moved on the sheet: R15
Changed lines of the file:
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@@
 <part name="D2" library="diode" deviceset="1N4446" device=""/>
 <part name="IC7" library="linear" deviceset="LM311" device="N"/>
-<part name="R8" library="resistor" deviceset="R-EU_" device="0309/V"/>
-<part name="R10" library="resistor" deviceset="R-TRIMM" device="4G/J"/>
+<part name="R8" library="resistor" deviceset="R-EU_" device="0309/V" value="3.3k"/>
+<part name="R10" library="resistor" deviceset="R-TRIMM" device="4G/J" value="2k"/>
 <part name="SUPPLY5" library="supply2" deviceset="+5V" device=""/>
 <part name="SUPPLY17" library="supply2" deviceset="GND" device=""/>
@@
 <part name="SUPPLY19" library="supply2" deviceset="-9V" device=""/>
 <part name="SUPPLY20" library="supply2" deviceset="+5V" device=""/>
-<part name="R11" library="resistor" deviceset="R-EU_" device="0309/V"/>
+<part name="R11" library="resistor" deviceset="R-EU_" device="0309/V" value="24k"/>
 <part name="SUPPLY21" library="supply2" deviceset="GND" device=""/>
-<part name="R13" library="resistor" deviceset="R-EU_" device="0309/V"/>
-<part name="R14" library="resistor" deviceset="R-EU_" device="0309/V"/>
+<part name="R13" library="resistor" deviceset="R-EU_" device="0309/V" value="330k"/>
+<part name="R14" library="resistor" deviceset="R-EU_" device="0309/V" value="33k"/>
 <part name="SUPPLY23" library="supply2" deviceset="GND" device=""/>
-<part name="R15" library="resistor" deviceset="R-EU_" device="0309/V"/>
+<part name="R15" library="resistor" deviceset="R-EU_" device="0309/V" value="2.2k"/>
 <part name="D3" library="diode" deviceset="1N4446" device="" value="1N4736_Zener_6.8V"/>
+<part name="R16" library="resistor" deviceset="R-EU_" device="0309/V" value="10k"/>
 </parts>
 <sheets>
@@
 <text x="-124.46" y="-10.16" size="1.778" layer="91">/-16V</text>
 <text x="46.736" y="46.99" size="1.9304" layer="91">zero pass signal</text>
-<text x="15.24" y="57.658" size="1.778" layer="91">hysterese</text>
+<text x="22.86" y="62.738" size="1.778" layer="91">hysterese</text>
 </plain>
 <instances>
@@
 <instance part="R14" gate="G$1" x="15.24" y="38.1" rot="R90"/>
 <instance part="SUPPLY23" gate="GND" x="15.24" y="30.48"/>
-<instance part="R15" gate="G$1" x="15.24" y="68.58"/>
+<instance part="R15" gate="G$1" x="20.32" y="71.12"/>
 <instance part="D3" gate="1" x="5.08" y="38.1" rot="R90"/>
+<instance part="R16" gate="G$1" x="40.64" y="66.04" smashed="yes">
+<attribute name="NAME" x="36.83" y="67.5386" size="1.778" layer="95"/>
+<attribute name="VALUE" x="39.37" y="62.738" size="1.778" layer="96"/>
+</instance>
 </instances>
 <busses>
@@
 <net name="N$22" class="0">
 <segment>
-<wire x1="10.16" y1="68.58" x2="10.16" y2="43.18" width="0.1524" layer="91"/>
-<wire x1="10.16" y1="43.18" x2="15.24" y2="43.18" width="0.1524" layer="91"/>
+<wire x1="10.16" y1="68.58" x2="5.08" y2="68.58" width="0.1524" layer="91"/>
+<wire x1="5.08" y1="68.58" x2="5.08" y2="40.64" width="0.1524" layer="91"/>
+<pinref part="D3" gate="1" pin="C"/>
 <pinref part="IC7" gate="A" pin="-IN"/>
 <wire x1="15.24" y1="43.18" x2="22.86" y2="43.18" width="0.1524" layer="91"/>
 <pinref part="R14" gate="G$1" pin="2"/>
+<wire x1="10.16" y1="43.18" x2="15.24" y2="43.18" width="0.1524" layer="91"/>
+<wire x1="10.16" y1="68.58" x2="10.16" y2="43.18" width="0.1524" layer="91"/>
 <pinref part="R15" gate="G$1" pin="1"/>
-<wire x1="10.16" y1="68.58" x2="5.08" y2="68.58" width="0.1524" layer="91"/>
-<wire x1="5.08" y1="68.58" x2="5.08" y2="40.64" width="0.1524" layer="91"/>
-<pinref part="D3" gate="1" pin="C"/>
+<wire x1="15.24" y1="71.12" x2="10.16" y2="71.12" width="0.1524" layer="91"/>
+<wire x1="10.16" y1="71.12" x2="10.16" y2="68.58" width="0.1524" layer="91"/>
 </segment>
 </net>
@@
 <net name="N$25" class="0">
 <segment>
-<pinref part="R10" gate="G$1" pin="S"/>
-<wire x1="45.72" y1="66.04" x2="12.7" y2="66.04" width="0.1524" layer="91"/>
+<wire x1="35.56" y1="66.04" x2="12.7" y2="66.04" width="0.1524" layer="91"/>
 <wire x1="12.7" y1="66.04" x2="12.7" y2="60.96" width="0.1524" layer="91"/>
 <wire x1="12.7" y1="60.96" x2="12.7" y2="48.26" width="0.1524" layer="91"/>
-<wire x1="12.7" y1="48.26" x2="22.86" y2="48.26" width="0.1524" layer="91"/>
-<pinref part="IC7" gate="A" pin="+IN"/>
 <pinref part="R13" gate="G$1" pin="1"/>
 <wire x1="15.24" y1="60.96" x2="12.7" y2="60.96" width="0.1524" layer="91"/>
+<pinref part="R16" gate="G$1" pin="1"/>
+<pinref part="IC7" gate="A" pin="+IN"/>
+<wire x1="12.7" y1="48.26" x2="22.86" y2="48.26" width="0.1524" layer="91"/>
 </segment>
 </net>
@@
 <wire x1="22.86" y1="93.98" x2="35.56" y2="93.98" width="0.1524" layer="91"/>
 <wire x1="35.56" y1="93.98" x2="35.56" y2="81.28" width="0.1524" layer="91"/>
-<wire x1="35.56" y1="81.28" x2="35.56" y2="68.58" width="0.1524" layer="91"/>
+<wire x1="35.56" y1="81.28" x2="35.56" y2="71.12" width="0.1524" layer="91"/>
 <wire x1="22.86" y1="81.28" x2="35.56" y2="81.28" width="0.1524" layer="91"/>
 <pinref part="D2" gate="1" pin="C"/>
 <pinref part="R15" gate="G$1" pin="2"/>
-<wire x1="20.32" y1="68.58" x2="35.56" y2="68.58" width="0.1524" layer="91"/>
+<wire x1="25.4" y1="71.12" x2="35.56" y2="71.12" width="0.1524" layer="91"/>
 </segment>
 </net>
@@
 </segment>
 </net>
+<net name="N$27" class="0">
+<segment>
+<pinref part="R10" gate="G$1" pin="S"/>
+<pinref part="R16" gate="G$1" pin="2"/>
+</segment>
+</net>
