File: eagle/joesTriac-2nd/powerBoard-2nd.sch (EAGLE design)
At the start: 44 parts, among them IC1 7809, IC2 7805, IC3 7909, IC5 7809, IC7 LM311N, J1 XF2E-0815-1, J2 XF2E-0815-1

Commit message: reg 0x schematics voltage save
Parts:
- removed R15: 2.2k, resistor:R-EU_0309/V
- added IC8: TLC251P, linear:TLC251P
- added J3: XF2E-0815-1, con-omron:XF2E-0815-1
- added R17: ~4k, resistor:R-EU_0309/V
Connections:
- new net N$24: B1.AC2, TR1.3
- new net N$30: IC8.-IN, IC8.OUT
- new net N$6: D1.C, D2.C, J3-3.MS
- net GND: now also R2.1
- net N$22: now also R17.1; no longer R15.1
- net N$28: now also R17.2; no longer D1.C, D2.C, R15.2
- net N$29: now also IC8.+IN
- net N$3: now also J3-1.MSV
- net N$4: no longer B1.AC2, TR1.3
Other:
- moved on the sheet: B1, C1, C10, C11, C2, C3, C4, C5, C6, C7, C8, C9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

Commit message: reg save
Parts:
- added J4: XF2E-0815-1, con-omron:XF2E-0815-1
- R17: value ~4k -> 2.2k
Connections:
- new net N$31: J4-3.MS, R10.S
- net GND: now also J4-1.MSV
- net N$27: no longer R10.S
Other:
- moved on the sheet: R10, R16, R8
Changed lines of the file:
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@@
 <part name="IC8" library="linear" deviceset="TLC251" device="P"/>
 <part name="J3" library="con-omron" deviceset="XF2*-08?" device="15-1" technology="E" value=""/>
-<part name="R17" library="resistor" deviceset="R-EU_" device="0309/V" value="~4k"/>
+<part name="R17" library="resistor" deviceset="R-EU_" device="0309/V" value="2.2k"/>
+<part name="J4" library="con-omron" deviceset="XF2*-08?" device="15-1" technology="E" value=""/>
 </parts>
 <sheets>
@@
 <instance part="D2" gate="1" x="7.62" y="81.28"/>
 <instance part="IC7" gate="A" x="25.4" y="45.72"/>
-<instance part="R8" gate="G$1" x="53.34" y="78.74" rot="R90"/>
-<instance part="R10" gate="G$1" x="53.34" y="68.58" rot="MR0"/>
-<instance part="SUPPLY5" gate="+5V" x="53.34" y="86.36"/>
-<instance part="SUPPLY17" gate="GND" x="53.34" y="63.5"/>
+<instance part="R8" gate="G$1" x="58.42" y="78.74" rot="R90"/>
+<instance part="R10" gate="G$1" x="58.42" y="68.58" rot="MR0"/>
+<instance part="SUPPLY5" gate="+5V" x="58.42" y="86.36"/>
+<instance part="SUPPLY17" gate="GND" x="58.42" y="60.96"/>
 <instance part="SUPPLY18" gate="G$1" x="22.86" y="55.88"/>
 <instance part="SUPPLY19" gate="G$1" x="20.32" y="33.02"/>
@@
 <instance part="SUPPLY23" gate="GND" x="10.16" y="27.94"/>
 <instance part="D3" gate="1" x="0" y="35.56" rot="R90"/>
-<instance part="R16" gate="G$1" x="38.1" y="68.58" smashed="yes">
-<attribute name="NAME" x="34.29" y="70.0786" size="1.778" layer="95"/>
-<attribute name="VALUE" x="36.83" y="65.278" size="1.778" layer="96"/>
+<instance part="R16" gate="G$1" x="35.56" y="68.58" smashed="yes">
+<attribute name="NAME" x="31.75" y="70.0786" size="1.778" layer="95"/>
+<attribute name="VALUE" x="34.29" y="65.278" size="1.778" layer="96"/>
 </instance>
 <instance part="IC8" gate="A" x="45.72" y="35.56"/>
@@
 <instance part="J3" gate="-3" x="27.94" y="78.74" rot="R180"/>
 <instance part="R17" gate="G$1" x="12.7" y="73.66"/>
+<instance part="J4" gate="-1" x="48.26" y="66.04" rot="R180"/>
+<instance part="J4" gate="-2" x="48.26" y="68.58" rot="R180"/>
+<instance part="J4" gate="-3" x="48.26" y="71.12" rot="R180"/>
 </instances>
 <busses>
@@
 <pinref part="R10" gate="G$1" pin="A"/>
 <pinref part="SUPPLY17" gate="GND" pin="GND"/>
-<wire x1="53.34" y1="66.04" x2="53.34" y2="63.5" width="0.1524" layer="91"/>
+<wire x1="58.42" y1="63.5" x2="55.88" y2="63.5" width="0.1524" layer="91"/>
+<wire x1="55.88" y1="63.5" x2="55.88" y2="66.04" width="0.1524" layer="91"/>
+<pinref part="J4" gate="-1" pin="MSV"/>
+<wire x1="55.88" y1="66.04" x2="50.8" y2="66.04" width="0.1524" layer="91"/>
 </segment>
 <segment>
@@
 <wire x1="5.08" y1="40.64" x2="10.16" y2="40.64" width="0.1524" layer="91"/>
 <wire x1="5.08" y1="71.12" x2="5.08" y2="43.18" width="0.1524" layer="91"/>
+<wire x1="5.08" y1="43.18" x2="5.08" y2="40.64" width="0.1524" layer="91"/>
+<pinref part="IC7" gate="A" pin="-IN"/>
+<wire x1="17.78" y1="43.18" x2="5.08" y2="43.18" width="0.1524" layer="91"/>
 <pinref part="R17" gate="G$1" pin="1"/>
-<wire x1="5.08" y1="43.18" x2="5.08" y2="40.64" width="0.1524" layer="91"/>
 <wire x1="7.62" y1="73.66" x2="5.08" y2="73.66" width="0.1524" layer="91"/>
 <wire x1="5.08" y1="73.66" x2="5.08" y2="71.12" width="0.1524" layer="91"/>
-<pinref part="IC7" gate="A" pin="-IN"/>
-<wire x1="17.78" y1="43.18" x2="5.08" y2="43.18" width="0.1524" layer="91"/>
 </segment>
 </net>
@@
 <pinref part="R8" gate="G$1" pin="1"/>
 <pinref part="R10" gate="G$1" pin="E"/>
-</segment>
-</net>
-<net name="N$25" class="0">
-<segment>
-<wire x1="7.62" y1="68.58" x2="7.62" y2="63.5" width="0.1524" layer="91"/>
-<pinref part="R16" gate="G$1" pin="1"/>
-<wire x1="33.02" y1="68.58" x2="7.62" y2="68.58" width="0.1524" layer="91"/>
-<pinref part="R13" gate="G$1" pin="1"/>
-<wire x1="12.7" y1="63.5" x2="7.62" y2="63.5" width="0.1524" layer="91"/>
-<wire x1="7.62" y1="63.5" x2="7.62" y2="48.26" width="0.1524" layer="91"/>
-<pinref part="IC7" gate="A" pin="+IN"/>
-<wire x1="10.16" y1="48.26" x2="12.7" y2="48.26" width="0.1524" layer="91"/>
-<wire x1="12.7" y1="48.26" x2="17.78" y2="48.26" width="0.1524" layer="91"/>
-<wire x1="7.62" y1="48.26" x2="10.16" y2="48.26" width="0.1524" layer="91"/>
 </segment>
 </net>
@@
 </segment>
 </net>
-<net name="N$27" class="0">
-<segment>
-<pinref part="R10" gate="G$1" pin="S"/>
-<pinref part="R16" gate="G$1" pin="2"/>
-<wire x1="43.18" y1="68.58" x2="48.26" y2="68.58" width="0.1524" layer="91"/>
-</segment>
-</net>
 <net name="N$30" class="0">
 <segment>
@@
 <net name="N$28" class="0">
 <segment>
+<wire x1="7.62" y1="68.58" x2="7.62" y2="63.5" width="0.1524" layer="91"/>
+<pinref part="R16" gate="G$1" pin="1"/>
+<wire x1="30.48" y1="68.58" x2="7.62" y2="68.58" width="0.1524" layer="91"/>
+<pinref part="R13" gate="G$1" pin="1"/>
+<wire x1="12.7" y1="63.5" x2="7.62" y2="63.5" width="0.1524" layer="91"/>
+<wire x1="7.62" y1="63.5" x2="7.62" y2="48.26" width="0.1524" layer="91"/>
+<pinref part="IC7" gate="A" pin="+IN"/>
+<wire x1="7.62" y1="48.26" x2="17.78" y2="48.26" width="0.1524" layer="91"/>
+</segment>
+</net>
+<net name="N$27" class="0">
+<segment>
+<pinref part="R16" gate="G$1" pin="2"/>
+<wire x1="40.64" y1="68.58" x2="48.26" y2="68.58" width="0.1524" layer="91"/>
+</segment>
+</net>
+<net name="N$31" class="0">
+<segment>
+<pinref part="R10" gate="G$1" pin="S"/>
+<wire x1="53.34" y1="68.58" x2="53.34" y2="71.12" width="0.1524" layer="91"/>
+<pinref part="J4" gate="-3" pin="MS"/>
+<wire x1="53.34" y1="71.12" x2="50.8" y2="71.12" width="0.1524" layer="91"/>
+</segment>
+</net>
+<net name="N$25" class="0">
+<segment>
 <wire x1="27.94" y1="76.2" x2="20.32" y2="76.2" width="0.1524" layer="91"/>
