File: eagle/joesTriac-2nd/cpuConnectionBoard.sch (EAGLE design)
At the start: 9 parts, among them IC1 24C01CP, J1 CN11, J2 CN9, J3 CN13, J4 CN14, Q1 2N4403

Commit message: reg save
Parts:
- added Q2: 2N4401, transistor-npn:2N4416
- added R3: 1k, resistor:R-EU_0309/12
- added R4: 47k, resistor:R-EU_0309/12
- R1: value (none) -> 1k
- R2: value (none) -> 47k
Connections:
- new net N$4: Q2.B, R1.2
- new net N$8: J2-9.MS, Q1.C, R4.2
- net GND: now also Q2.E, R4.1
- net N$3: now also R3.2; no longer R1.2
- net N$5: now also Q2.C, R3.1; no longer Q1.C
Other:
- note removed: "on stm32 opendrain-pullup port"
- moved on the sheet: R1
Changed lines of the file:
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@@
 <part name="J4" library="con-omron" deviceset="XF2*-08?" device="15-1" technology="E" value="CN14"/>
 <part name="Q1" library="transistor-pnp" deviceset="2N4902" device="" value="2N4403"/>
-<part name="R1" library="resistor" deviceset="R-EU_" device="0309/12"/>
-<part name="R2" library="resistor" deviceset="R-EU_" device="0309/12"/>
+<part name="R1" library="resistor" deviceset="R-EU_" device="0309/12" value="1k"/>
+<part name="R2" library="resistor" deviceset="R-EU_" device="0309/12" value="47k"/>
+<part name="Q2" library="transistor-npn" deviceset="2N4416" device="" value="2N4401"/>
+<part name="R3" library="resistor" deviceset="R-EU_" device="0309/12" value="1k"/>
+<part name="SUPPLY7" library="supply2" deviceset="GND" device=""/>
+<part name="R4" library="resistor" deviceset="R-EU_" device="0309/12" value="47k"/>
 </parts>
 <sheets>
@@
 <text x="88.9" y="0" size="1.778" layer="91">out</text>
 <text x="-15.24" y="48.26" size="1.778" layer="91">PH6</text>
-<text x="55.88" y="33.02" size="1.778" layer="91">on stm32 opendrain-pullup port</text>
-<text x="119.38" y="50.8" size="1.778" layer="91">triac trigger</text>
+<text x="124.46" y="38.1" size="1.778" layer="91">triac trigger</text>
 </plain>
 <instances>
@@
 <instance part="J4" gate="-6" x="78.74" y="-43.18"/>
 <instance part="Q1" gate="A" x="114.3" y="58.42"/>
-<instance part="R1" gate="G$1" x="99.06" y="30.48"/>
+<instance part="R1" gate="G$1" x="73.66" y="30.48"/>
 <instance part="R2" gate="G$1" x="93.98" y="66.04" rot="R90"/>
+<instance part="Q2" gate="G$1" x="81.28" y="30.48"/>
+<instance part="R3" gate="G$1" x="93.98" y="48.26"/>
+<instance part="SUPPLY7" gate="GND" x="104.14" y="15.24"/>
+<instance part="R4" gate="G$1" x="116.84" y="27.94" rot="R90"/>
 </instances>
 <busses>
@@
 <wire x1="73.66" y1="-10.16" x2="58.42" y2="-10.16" width="0.1524" layer="91"/>
 <pinref part="J1" gate="-7" pin="MS"/>
-<wire x1="58.42" y1="-10.16" x2="48.26" y2="-10.16" width="0.1524" layer="91"/>
 <wire x1="76.2" y1="-15.24" x2="73.66" y2="-15.24" width="0.1524" layer="91"/>
 <wire x1="73.66" y1="-15.24" x2="73.66" y2="-10.16" width="0.1524" layer="91"/>
 <pinref part="SUPPLY5" gate="GND" pin="GND"/>
 <junction x="58.42" y="-10.16"/>
+<wire x1="58.42" y1="-10.16" x2="25.4" y2="-10.16" width="0.1524" layer="91"/>
+<wire x1="25.4" y1="-10.16" x2="25.4" y2="17.78" width="0.1524" layer="91"/>
+<wire x1="25.4" y1="17.78" x2="83.82" y2="17.78" width="0.1524" layer="91"/>
+<pinref part="Q2" gate="G$1" pin="E"/>
+<wire x1="83.82" y1="17.78" x2="104.14" y2="17.78" width="0.1524" layer="91"/>
+<wire x1="104.14" y1="17.78" x2="116.84" y2="17.78" width="0.1524" layer="91"/>
+<wire x1="83.82" y1="25.4" x2="83.82" y2="17.78" width="0.1524" layer="91"/>
+<pinref part="SUPPLY7" gate="GND" pin="GND"/>
+<junction x="104.14" y="17.78"/>
+<pinref part="R4" gate="G$1" pin="1"/>
+<wire x1="116.84" y1="22.86" x2="116.84" y2="17.78" width="0.1524" layer="91"/>
 </segment>
 <segment>
@@
 <wire x1="-17.78" y1="45.72" x2="-10.16" y2="45.72" width="0.1524" layer="91"/>
 <wire x1="-10.16" y1="45.72" x2="-10.16" y2="30.48" width="0.1524" layer="91"/>
-<wire x1="-10.16" y1="30.48" x2="93.98" y2="30.48" width="0.1524" layer="91"/>
+<wire x1="-10.16" y1="30.48" x2="68.58" y2="30.48" width="0.1524" layer="91"/>
 <pinref part="R1" gate="G$1" pin="1"/>
 </segment>
@@
 <segment>
 <pinref part="Q1" gate="A" pin="B"/>
-<wire x1="111.76" y1="58.42" x2="106.68" y2="58.42" width="0.1524" layer="91"/>
-<wire x1="106.68" y1="58.42" x2="106.68" y2="30.48" width="0.1524" layer="91"/>
-<wire x1="106.68" y1="30.48" x2="104.14" y2="30.48" width="0.1524" layer="91"/>
-<pinref part="R1" gate="G$1" pin="2"/>
 <pinref part="R2" gate="G$1" pin="1"/>
 <wire x1="93.98" y1="60.96" x2="93.98" y2="58.42" width="0.1524" layer="91"/>
 <wire x1="93.98" y1="58.42" x2="106.68" y2="58.42" width="0.1524" layer="91"/>
+<pinref part="R3" gate="G$1" pin="2"/>
+<wire x1="106.68" y1="58.42" x2="111.76" y2="58.42" width="0.1524" layer="91"/>
+<wire x1="99.06" y1="48.26" x2="106.68" y2="48.26" width="0.1524" layer="91"/>
+<wire x1="106.68" y1="48.26" x2="106.68" y2="58.42" width="0.1524" layer="91"/>
+</segment>
+</net>
+<net name="N$4" class="0">
+<segment>
+<pinref part="R1" gate="G$1" pin="2"/>
+<pinref part="Q2" gate="G$1" pin="B"/>
 </segment>
 </net>
 <net name="N$5" class="0">
 <segment>
+<pinref part="Q2" gate="G$1" pin="C"/>
+<wire x1="83.82" y1="35.56" x2="83.82" y2="48.26" width="0.1524" layer="91"/>
+<pinref part="R3" gate="G$1" pin="1"/>
+<wire x1="83.82" y1="48.26" x2="88.9" y2="48.26" width="0.1524" layer="91"/>
+</segment>
+</net>
+<net name="N$8" class="0">
+<segment>
 <pinref part="Q1" gate="A" pin="C"/>
-<wire x1="116.84" y1="53.34" x2="116.84" y2="48.26" width="0.1524" layer="91"/>
-<wire x1="116.84" y1="48.26" x2="139.7" y2="48.26" width="0.1524" layer="91"/>
-</segment>
-</net>
+<wire x1="116.84" y1="53.34" x2="116.84" y2="38.1" width="0.1524" layer="91"/>
+<pinref part="R4" gate="G$1" pin="2"/>
+<wire x1="116.84" y1="38.1" x2="116.84" y2="33.02" width="0.1524" layer="91"/>
+<wire x1="116.84" y1="38.1" x2="121.92" y2="38.1" width="0.1524" layer="91"/>
+<wire x1="121.92" y1="38.1" x2="121.92" y2="-17.78" width="0.1524" layer="91"/>
+<pinref part="J2" gate="-9" pin="MS"/>
+<wire x1="121.92" y1="-17.78" x2="157.48" y2="-17.78" width="0.1524" layer="91"/>
+</segment>
+</net>
