File: eagle/joesTriac-2nd/AmmeterBoard-2nd.sch (EAGLE design)
At the start: 36 parts, among them IC10 LM317MB, IC12 LM337, IC13 TLC251P, IC14 TLC251P, IC15 TLC251P, IC6 TLC251P, IC7 ACS758ECB-200B-PFF-T, IC8 X9C104P, X1 1, X2 2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

Commit message: reg save
Parts:
- removed X3: 1, con-phoenix-350:1751251
- added JP1, JP3, JP4: (no value), jumper:JP2E
- added X4, X5: (no value), con-phoenix-254:MPT6
- added X6: 1751264, con-phoenix-350:1751264
Connections:
- removed net N$10: IC7.VOUT, X3-2.K
- new net GND1: C11.+, C6.-
- new net N$13: JP4.2
- new net N$15: JP3.2
- new net N$3: X6-4.K
- new net N$4: IC7.VCC, X6-2.K
- new net N$5: IC7.VOUT, X6-3.K
- new net N$6: X6-1.K
- new net N$9: JP1.2
- net +4.1V: now also X4-1.1
- net +9V: now also X4-3.1
- net -4.1V: now also X4-2.1
- net -9V: now also X4-4.1
- net GND: no longer C11.+, C6.-
- net N$26: now also X5-1.1
- net N$31: now also X5-2.1
- net N$32: now also X5-3.1
- net SENS+: no longer IC7.VCC, X3-1.K
- net SENS-: no longer IC7.GND, X3-3.K
Other:
- note added: "all jumpers 1-2 or 2-3"
- note added: "gnd_in/out"
- note added: "to cpuboard"
- note added: "to powerboard"

Commit message: reg save
Connections:
- new net N$10: IC8.U/D, X5-2.1
- net N$31: now also X5-3.1; no longer X5-2.1
- net N$32: now also X5-4.1; no longer X5-3.1
Changed lines of the file:
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@@
 <net name="N$32" class="0">
 <segment>
-<wire x1="167.64" y1="2.54" x2="152.4" y2="2.54" width="0.1524" layer="91"/>
+<wire x1="180.34" y1="2.54" x2="152.4" y2="2.54" width="0.1524" layer="91"/>
 <wire x1="152.4" y1="2.54" x2="149.86" y2="2.54" width="0.1524" layer="91"/>
 <pinref part="IC8" gate="1" pin="!CS"/>
 <junction x="152.4" y="2.54"/>
-<wire x1="167.64" y1="2.54" x2="167.64" y2="5.08" width="0.1524" layer="91"/>
-<wire x1="167.64" y1="5.08" x2="193.04" y2="5.08" width="0.1524" layer="91"/>
-<pinref part="X5" gate="-3" pin="1"/>
-<wire x1="193.04" y1="5.08" x2="195.58" y2="5.08" width="0.1524" layer="91"/>
-<junction x="193.04" y="5.08"/>
+<wire x1="180.34" y1="2.54" x2="180.34" y2="0" width="0.1524" layer="91"/>
+<pinref part="X5" gate="-4" pin="1"/>
+<wire x1="180.34" y1="0" x2="193.04" y2="0" width="0.1524" layer="91"/>
 </segment>
 </net>
 <net name="N$31" class="0">
 <segment>
-<wire x1="162.56" y1="5.08" x2="152.4" y2="5.08" width="0.1524" layer="91"/>
 <pinref part="IC8" gate="1" pin="!INC"/>
 <wire x1="152.4" y1="5.08" x2="149.86" y2="5.08" width="0.1524" layer="91"/>
 <junction x="152.4" y="5.08"/>
-<wire x1="162.56" y1="5.08" x2="162.56" y2="10.16" width="0.1524" layer="91"/>
-<pinref part="X5" gate="-2" pin="1"/>
-<wire x1="162.56" y1="10.16" x2="193.04" y2="10.16" width="0.1524" layer="91"/>
+<pinref part="X5" gate="-3" pin="1"/>
+<wire x1="193.04" y1="5.08" x2="195.58" y2="5.08" width="0.1524" layer="91"/>
+<wire x1="152.4" y1="5.08" x2="193.04" y2="5.08" width="0.1524" layer="91"/>
 </segment>
 </net>
@@
 </segment>
 </net>
+<net name="N$10" class="0">
+<segment>
+<pinref part="IC8" gate="1" pin="U/D"/>
+<wire x1="152.4" y1="7.62" x2="180.34" y2="7.62" width="0.1524" layer="91"/>
+<wire x1="180.34" y1="7.62" x2="180.34" y2="10.16" width="0.1524" layer="91"/>
+<pinref part="X5" gate="-2" pin="1"/>
+<wire x1="180.34" y1="10.16" x2="193.04" y2="10.16" width="0.1524" layer="91"/>
+</segment>
+</net>

Commit message: reg save
Connections:
- net GND: now also X4-5.1
Other:
- moved on the sheet: X4-1, X4-2, X4-3, X4-4, X4-5, X4-6
Changed lines of the file:
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@@
 <part name="SUPPLY8" library="supply2" deviceset="-4.1V" device="" value="-2.5V"/>
 <part name="SUPPLY9" library="supply2" deviceset="GND" device=""/>
+<part name="SUPPLY18" library="supply2" deviceset="GND" device=""/>
 </parts>
 <sheets>
@@
 <text x="-35.56" y="-33.02" size="1.778" layer="91">SENS+, SENS- are connected to sensor (see sheet 1)</text>
 <text x="106.68" y="33.02" size="1.778" layer="91">SENSSIG is connected to sensor</text>
-<text x="182.88" y="111.76" size="3.302" layer="91">to powerboard</text>
+<text x="182.88" y="116.84" size="3.302" layer="91">to powerboard</text>
 <text x="185.42" y="22.86" size="3.302" layer="91">to cpuboard</text>
 <text x="-12.7" y="101.6" size="1.778" layer="91">gnd_in/out</text>
@@
 <instance part="SUPPLY31" gate="G$1" x="17.78" y="-30.48" rot="MR0"/>
 <instance part="C11" gate="G$1" x="-27.94" y="-10.16"/>
-<instance part="X4" gate="-1" x="195.58" y="101.6"/>
-<instance part="X4" gate="-2" x="195.58" y="96.52"/>
-<instance part="X4" gate="-3" x="195.58" y="91.44"/>
-<instance part="X4" gate="-4" x="195.58" y="86.36"/>
-<instance part="X4" gate="-5" x="195.58" y="81.28"/>
-<instance part="X4" gate="-6" x="195.58" y="76.2"/>
+<instance part="X4" gate="-1" x="195.58" y="106.68"/>
+<instance part="X4" gate="-2" x="195.58" y="101.6"/>
+<instance part="X4" gate="-3" x="195.58" y="96.52"/>
+<instance part="X4" gate="-4" x="195.58" y="91.44"/>
+<instance part="X4" gate="-5" x="195.58" y="86.36"/>
+<instance part="X4" gate="-6" x="195.58" y="81.28"/>
 <instance part="X5" gate="-1" x="195.58" y="15.24"/>
 <instance part="X5" gate="-2" x="195.58" y="10.16"/>
@@
 <instance part="X5" gate="-5" x="195.58" y="-5.08"/>
 <instance part="X5" gate="-6" x="195.58" y="-10.16"/>
-<instance part="SUPPLY1" gate="P" x="187.96" y="104.14" rot="MR0"/>
-<instance part="SUPPLY2" gate="P" x="165.1" y="101.6" rot="MR180"/>
-<instance part="SUPPLY3" gate="G$1" x="177.8" y="93.98"/>
-<instance part="SUPPLY4" gate="G$1" x="165.1" y="91.44"/>
+<instance part="SUPPLY1" gate="P" x="187.96" y="109.22" rot="MR0"/>
+<instance part="SUPPLY2" gate="P" x="165.1" y="106.68" rot="MR180"/>
+<instance part="SUPPLY3" gate="G$1" x="177.8" y="99.06"/>
+<instance part="SUPPLY4" gate="G$1" x="160.02" y="96.52"/>
 <instance part="SUPPLY5" gate="G$1" x="-15.24" y="-2.54"/>
 <instance part="X6" gate="-1" x="0" y="99.06"/>
@@
 <instance part="SUPPLY8" gate="P" x="12.7" y="45.72" rot="MR180"/>
 <instance part="SUPPLY9" gate="GND" x="33.02" y="45.72"/>
+<instance part="SUPPLY18" gate="GND" x="165.1" y="88.9"/>
 </instances>
 <busses>
@@
 <pinref part="SUPPLY9" gate="GND" pin="GND"/>
 <wire x1="30.48" y1="48.26" x2="33.02" y2="48.26" width="0.1524" layer="91"/>
+</segment>
+<segment>
+<pinref part="X4" gate="-5" pin="1"/>
+<wire x1="193.04" y1="86.36" x2="172.72" y2="86.36" width="0.1524" layer="91"/>
+<wire x1="172.72" y1="86.36" x2="172.72" y2="91.44" width="0.1524" layer="91"/>
+<pinref part="SUPPLY18" gate="GND" pin="GND"/>
+<wire x1="172.72" y1="91.44" x2="165.1" y2="91.44" width="0.1524" layer="91"/>
 </segment>
 </net>
@@
 <segment>
 <pinref part="X4" gate="-3" pin="1"/>
-<wire x1="193.04" y1="91.44" x2="177.8" y2="91.44" width="0.1524" layer="91"/>
+<wire x1="193.04" y1="96.52" x2="177.8" y2="96.52" width="0.1524" layer="91"/>
 <pinref part="SUPPLY3" gate="G$1" pin="+9V"/>
 </segment>
@@
 <segment>
 <pinref part="X4" gate="-4" pin="1"/>
-<wire x1="193.04" y1="86.36" x2="175.26" y2="86.36" width="0.1524" layer="91"/>
-<wire x1="175.26" y1="86.36" x2="175.26" y2="93.98" width="0.1524" layer="91"/>
-<wire x1="175.26" y1="93.98" x2="165.1" y2="93.98" width="0.1524" layer="91"/>
+<wire x1="193.04" y1="91.44" x2="175.26" y2="91.44" width="0.1524" layer="91"/>
+<wire x1="175.26" y1="91.44" x2="175.26" y2="99.06" width="0.1524" layer="91"/>
+<wire x1="175.26" y1="99.06" x2="160.02" y2="99.06" width="0.1524" layer="91"/>
 <pinref part="SUPPLY4" gate="G$1" pin="-9V"/>
 </segment>
@@
 </segment>
 <segment>
-<wire x1="195.58" y1="96.52" x2="193.04" y2="96.52" width="0.1524" layer="91"/>
-<wire x1="193.04" y1="96.52" x2="182.88" y2="96.52" width="0.1524" layer="91"/>
-<wire x1="182.88" y1="96.52" x2="182.88" y2="104.14" width="0.1524" layer="91"/>
+<wire x1="195.58" y1="101.6" x2="193.04" y2="101.6" width="0.1524" layer="91"/>
+<wire x1="193.04" y1="101.6" x2="182.88" y2="101.6" width="0.1524" layer="91"/>
+<wire x1="182.88" y1="101.6" x2="182.88" y2="109.22" width="0.1524" layer="91"/>
 <pinref part="SUPPLY2" gate="P" pin="-4.1V"/>
-<wire x1="182.88" y1="104.14" x2="165.1" y2="104.14" width="0.1524" layer="91"/>
+<wire x1="182.88" y1="109.22" x2="165.1" y2="109.22" width="0.1524" layer="91"/>
 <pinref part="X4" gate="-2" pin="1"/>
-<junction x="193.04" y="96.52"/>
+<junction x="193.04" y="101.6"/>
 </segment>
 <segment>
@@
 <segment>
 <pinref part="X4" gate="-1" pin="1"/>
-<wire x1="193.04" y1="101.6" x2="187.96" y2="101.6" width="0.1524" layer="91"/>
-<wire x1="187.96" y1="101.6" x2="187.96" y2="104.14" width="0.1524" layer="91"/>
+<wire x1="193.04" y1="106.68" x2="187.96" y2="106.68" width="0.1524" layer="91"/>
+<wire x1="187.96" y1="106.68" x2="187.96" y2="109.22" width="0.1524" layer="91"/>
 <pinref part="SUPPLY1" gate="P" pin="+4.1V"/>
-<junction x="187.96" y="101.6"/>
-</segment>
-<segment>
+<junction x="187.96" y="106.68"/>
+</segment>
+<segment>

Commit message: reg save
Parts:
- removed C11: 10u, resistor:CPOL-EUE5-10.5
- removed C6: 100u, resistor:CPOL-EUE5-10.5
- removed IC10: LM317MB, v-reg:LM317MB
- removed IC12: LM337, v-reg:LM337TL
- removed IC13, IC14, IC15: TLC251P, linear:TLC251P
- removed IC8: X9C104P, pot-xicor:X9C102P
- removed JP1, JP2, JP3, JP4: (no value), jumper:JP2E
- removed R15: 100k, resistor:R-EU_0207/10
- removed R17, R24: 10k, resistor:R-EU_0207/10
- removed R23: 10k, pot:TRIM_EU-B90P
- removed R25, R26: 20k, resistor:R-EU_0207/10
- removed R27: 1k, resistor:R-EU_0207/10
- removed R28, R29: 220, resistor:R-EU_0207/10
- removed R30, R31: 240, resistor:R-EU_0207/10
- added IC2, IC3: TLC251P, linear:TLC251P
- added R1, R2: 10k, resistor:R-EU_0207/10
- added R3: 50k, pot:TRIM_EU-B90P
- added SG1: F/EE21P, buzzer:F/EE21P
- added T1: 2N3441, transistor:2N3441
Connections:
- removed net GND1: C11.+, C6.-
- removed net N$15: JP3.2
- removed net N$24: IC1.BOUT
- removed net N$32: IC8.!CS, X5-4.1
- removed net N$33: IC13.+IN, R23.S
- removed net N$34: R17.1, R23.A
- removed net N$35: R23.E, R24.2
- removed net N$36: IC13.-IN, IC13.OUT, R26.1
- removed net N$37: IC14.+IN, IC8.W
- removed net N$38: IC14.-IN, IC14.OUT, R25.1
- removed net N$39: R29.2, R30.1
- removed net N$40: IC15.OUT, JP2.2, R27.2
- removed net N$41: IC15.-IN, R25.2, R26.2, R27.1
- removed net N$42: IC10.ADJ, R28.2, R29.1
- removed net SENS+: C6.+, IC10.OUT, R28.1
- removed net SENS-: C11.-, IC12.ADJ, IC12.OUT, R30.2, R31.1, R31.2
- new net +5V: SG1.1, X4-6.1
- new net N$11: IC2.-IN, IC2.OUT, R2.2
- new net N$7: SG1.2, T1.C
- net +4.1V: no longer IC8.H, IC8.VCC
- net +9V: no longer IC10.IN, R17.2
- net -4.1V: no longer IC8.GND, IC8.L
- net -9V: no longer IC12.IN, R24.1
- net GND: now also IC3.+IN, T1.E; no longer IC15.+IN, JP2.1, R15.1
- net N$1: now also R3.E, X6-3.K; no longer JP2.3
- net N$10: now also R1.1; no longer IC8.U/D
- net N$13: now also IC3.-IN, R2.1, R3.S; no longer JP4.2
- net N$26: no longer R15.2
- net N$31: no longer IC8.!INC
- net N$5: now also IC2.+IN; no longer X6-3.K
- net N$9: now also R1.2, T1.B; no longer JP1.2
Other:
- note removed: "SENSSIG is connected to sensor"
- note removed: "all jumpers 1-2 or 2-3"

Commit message: reg save
Parts:
- added IC4: INA118P, burr-brown:INA118P
Changed lines of the file:
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@@
 <part name="R3" library="pot" deviceset="TRIM_EU-" device="B90P" value="50k"/>
 <part name="SUPPLY20" library="supply2" deviceset="GND" device=""/>
+<part name="IC4" library="burr-brown" deviceset="INA118" device="P"/>
 </parts>
 <sheets>
@@
 <instance part="R3" gate="1" x="10.16" y="22.86" rot="R270"/>
 <instance part="SUPPLY20" gate="GND" x="10.16" y="2.54"/>
+<instance part="IC4" gate="G$1" x="7.62" y="-17.78"/>
 </instances>
 <busses>

Commit message: reg save
Parts:
- removed IC2, IC3: TLC251P, linear:TLC251P
- removed R3: 50k, pot:TRIM_EU-B90P
- R2: value 10k -> 100k; device resistor:R-EU_0207/10 -> pot:TRIM_EU-B90P
Connections:
- net +9V: now also IC4.V+
- net -9V: now also IC4.V-
- net GND: now also IC4.REF; no longer IC3.+IN
- net N$1: now also IC4.OUT; no longer R3.E
- net N$11: now also IC4.RG@1, R2.A; no longer IC2.-IN, IC2.OUT, R2.2
- net N$13: now also IC4.RG, R2.S; no longer IC3.-IN, R2.1, R3.S
- net N$5: now also IC4.-IN; no longer IC2.+IN
Other:
- note added: "vss"
- moved on the sheet: IC4
Changed lines of the file:
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@@
 <part name="R1" library="resistor" deviceset="R-EU_" device="0207/10" value="10k"/>
 <part name="SUPPLY19" library="supply2" deviceset="GND" device=""/>
-<part name="IC2" library="linear" deviceset="TLC251" device="P"/>
-<part name="IC3" library="linear" deviceset="TLC251" device="P"/>
-<part name="R2" library="resistor" deviceset="R-EU_" device="0207/10" value="10k"/>
-<part name="R3" library="pot" deviceset="TRIM_EU-" device="B90P" value="50k"/>
 <part name="SUPPLY20" library="supply2" deviceset="GND" device=""/>
 <part name="IC4" library="burr-brown" deviceset="INA118" device="P"/>
+<part name="R2" library="pot" deviceset="TRIM_EU-" device="B90P" value="100k"/>
+<part name="SUPPLY21" library="supply2" deviceset="+9V" device=""/>
+<part name="SUPPLY22" library="supply2" deviceset="-9V" device=""/>
+<part name="SUPPLY23" library="supply2" deviceset="GND" device=""/>
 </parts>
 <sheets>
@@
 <text x="185.42" y="22.86" size="3.302" layer="91">to cpuboard</text>
 <text x="-12.7" y="101.6" size="1.778" layer="91">gnd_in/out</text>
+<text x="-17.78" y="78.74" size="2.54" layer="91">vss</text>
 </plain>
 <instances>
@@
 <instance part="R1" gate="G$1" x="167.64" y="0" rot="R180"/>
 <instance part="SUPPLY19" gate="GND" x="142.24" y="-10.16"/>
-<instance part="IC2" gate="A" x="-15.24" y="15.24"/>
-<instance part="IC3" gate="A" x="22.86" y="12.7" rot="MR180"/>
-<instance part="R2" gate="G$1" x="2.54" y="15.24" rot="R180"/>
-<instance part="R3" gate="1" x="10.16" y="22.86" rot="R270"/>
-<instance part="SUPPLY20" gate="GND" x="10.16" y="2.54"/>
-<instance part="IC4" gate="G$1" x="7.62" y="-17.78"/>
+<instance part="SUPPLY20" gate="GND" x="-27.94" y="-10.16"/>
+<instance part="IC4" gate="G$1" x="-2.54" y="5.08"/>
+<instance part="R2" gate="1" x="-27.94" y="10.16"/>
+<instance part="SUPPLY21" gate="G$1" x="25.4" y="2.54"/>
+<instance part="SUPPLY22" gate="G$1" x="25.4" y="-10.16"/>
+<instance part="SUPPLY23" gate="GND" x="17.78" y="5.08"/>
 </instances>
 <busses>
@@
 </segment>
 <segment>
-<pinref part="IC3" gate="A" pin="+IN"/>
-<wire x1="15.24" y1="10.16" x2="10.16" y2="10.16" width="0.1524" layer="91"/>
-<wire x1="10.16" y1="10.16" x2="10.16" y2="5.08" width="0.1524" layer="91"/>
+<wire x1="-20.32" y1="0" x2="-27.94" y2="0" width="0.1524" layer="91"/>
+<wire x1="-27.94" y1="0" x2="-27.94" y2="-7.62" width="0.1524" layer="91"/>
 <pinref part="SUPPLY20" gate="GND" pin="GND"/>
+</segment>
+<segment>
+<pinref part="IC4" gate="G$1" pin="REF"/>
+<wire x1="12.7" y1="2.54" x2="12.7" y2="7.62" width="0.1524" layer="91"/>
+<pinref part="SUPPLY23" gate="GND" pin="GND"/>
+<wire x1="12.7" y1="7.62" x2="17.78" y2="7.62" width="0.1524" layer="91"/>
 </segment>
 </net>
@@
 <pinref part="SUPPLY3" gate="G$1" pin="+9V"/>
 </segment>
+<segment>
+<pinref part="IC4" gate="G$1" pin="V+"/>
+<pinref part="SUPPLY21" gate="G$1" pin="+9V"/>
+<wire x1="12.7" y1="0" x2="25.4" y2="0" width="0.1524" layer="91"/>
+</segment>
 </net>
 <net name="-9V" class="0">
@@
 <wire x1="175.26" y1="99.06" x2="160.02" y2="99.06" width="0.1524" layer="91"/>
 <pinref part="SUPPLY4" gate="G$1" pin="-9V"/>
+</segment>
+<segment>
+<pinref part="IC4" gate="G$1" pin="V-"/>
+<wire x1="12.7" y1="-5.08" x2="25.4" y2="-5.08" width="0.1524" layer="91"/>
+<pinref part="SUPPLY22" gate="G$1" pin="-9V"/>
+<wire x1="25.4" y1="-5.08" x2="25.4" y2="-7.62" width="0.1524" layer="91"/>
 </segment>
 </net>
@@
 </segment>
 </net>
-<net name="N$11" class="0">
-<segment>
-<pinref part="IC2" gate="A" pin="OUT"/>
-<wire x1="-7.62" y1="15.24" x2="-2.54" y2="15.24" width="0.1524" layer="91"/>
-<wire x1="-2.54" y1="15.24" x2="-2.54" y2="5.08" width="0.1524" layer="91"/>
-<wire x1="-2.54" y1="5.08" x2="-25.4" y2="5.08" width="0.1524" layer="91"/>
-<wire x1="-25.4" y1="5.08" x2="-25.4" y2="12.7" width="0.1524" layer="91"/>
-<pinref part="IC2" gate="A" pin="-IN"/>
-<wire x1="-25.4" y1="12.7" x2="-22.86" y2="12.7" width="0.1524" layer="91"/>
-<pinref part="R2" gate="G$1" pin="2"/>
-<junction x="-2.54" y="15.24"/>
-</segment>
-</net>
-<net name="N$13" class="0">
-<segment>
-<pinref part="R2" gate="G$1" pin="1"/>
-<wire x1="7.62" y1="15.24" x2="10.16" y2="15.24" width="0.1524" layer="91"/>
-<pinref part="R3" gate="1" pin="S"/>
-<wire x1="10.16" y1="17.78" x2="10.16" y2="15.24" width="0.1524" layer="91"/>
-<pinref part="IC3" gate="A" pin="-IN"/>
-<wire x1="10.16" y1="15.24" x2="15.24" y2="15.24" width="0.1524" layer="91"/>
-</segment>
-</net>
 <net name="N$5" class="0">
 <segment>
@@
 <wire x1="-7.62" y1="76.2" x2="-7.62" y2="50.8" width="0.1524" layer="91"/>
 <wire x1="-25.4" y1="50.8" x2="-25.4" y2="17.78" width="0.1524" layer="91"/>
-<pinref part="IC2" gate="A" pin="+IN"/>
-<wire x1="-25.4" y1="17.78" x2="-22.86" y2="17.78" width="0.1524" layer="91"/>
 <wire x1="-25.4" y1="50.8" x2="-7.62" y2="50.8" width="0.1524" layer="91"/>
+<pinref part="IC4" gate="G$1" pin="-IN"/>
+<wire x1="-25.4" y1="17.78" x2="-20.32" y2="17.78" width="0.1524" layer="91"/>
 </segment>
 </net>
@@
 <wire x1="-5.08" y1="76.2" x2="-5.08" y2="33.02" width="0.1524" layer="91"/>
 <wire x1="-5.08" y1="33.02" x2="35.56" y2="33.02" width="0.1524" layer="91"/>
-<wire x1="35.56" y1="33.02" x2="35.56" y2="22.86" width="0.1524" layer="91"/>
-<pinref part="R3" gate="1" pin="E"/>
-<wire x1="15.24" y1="22.86" x2="35.56" y2="22.86" width="0.1524" layer="91"/>
-<wire x1="35.56" y1="22.86" x2="35.56" y2="12.7" width="0.1524" layer="91"/>
-<wire x1="35.56" y1="12.7" x2="27.94" y2="12.7" width="0.1524" layer="91"/>
-</segment>
-</net>
+<wire x1="35.56" y1="33.02" x2="35.56" y2="10.16" width="0.1524" layer="91"/>
+<pinref part="IC4" gate="G$1" pin="OUT"/>
+<wire x1="12.7" y1="10.16" x2="35.56" y2="10.16" width="0.1524" layer="91"/>
+</segment>
+</net>
+<net name="N$11" class="0">
+<segment>
+<pinref part="IC4" gate="G$1" pin="RG@1"/>
+<pinref part="R2" gate="1" pin="A"/>
+<wire x1="-20.32" y1="5.08" x2="-27.94" y2="5.08" width="0.1524" layer="91"/>
+</segment>
+</net>
+<net name="N$13" class="0">
+<segment>
+<pinref part="IC4" gate="G$1" pin="RG"/>
+<wire x1="-20.32" y1="12.7" x2="-22.86" y2="12.7" width="0.1524" layer="91"/>
+<pinref part="R2" gate="1" pin="S"/>
+<wire x1="-22.86" y1="12.7" x2="-22.86" y2="10.16" width="0.1524" layer="91"/>
+</segment>
+</net>

Commit message: reg save
Parts:
- added IC2: TLC251P, linear:TLC251P
- added IC3: TLC251_or_311, linear:TLC251P
- added R3: approx._1k, resistor:R-EU_0207/10
- added R4: approx_50k, resistor:R-EU_0207/10
Connections:
- removed net N$47: R9.A, R9.S
- new net N$14: IC2.+IN
- new net N$15: IC2.-IN, IC2.OUT, IC3.+IN, R9.A, R9.S
- new net N$16: IC3.OUT, R3.2, X5-6.1
- new net N$17: IC3.-IN, R3.1, R4.1
- net +9V: now also IC2.V+
- net -9V: now also IC2.V-
- net GND: now also IC4.+IN, R4.2
- net N$3: now also IC7.GND
Other:
- note added: "AD637"
- note added: "WIP - work in progress in 637 part"
- note added: "currentZeroPass"
- note added: "important: isr only if moving towards GND"
- note removed: "AD536"
- moved on the sheet: IC4, R2, X6-1, X6-2, X6-3, X6-4
