File: eagle/joesTriac-2nd/triacBoard.sch (EAGLE design)
At the start: 12 parts, among them IC2 LM311N, X1 87832-06

Commit message: reg save
Parts:
- removed IC1: (no value), atmel-new:ATTINY4414P3
- removed IC2: LM311N, linear:LM311N
- removed JP1, JP2: (no value), jumper:JP2E
- removed SL1: (no value), con-amp-quick:M06
- added -: BTA24-800, triac:BTA24-800
- added F1: FUSE 1A, fuse:FUSESH22,5
- added F3: FUSE 16A, fuse:FUSESH22,5
- added OK1: TIL196, optocoupler:TIL196
- added Q1: 2N2222A, transistor-npn:2N2222A
- added R6: 10k, resistor:R-EU_0207/15
- added R7: 70k, resistor:R-EU_0207/15
- added R8: 1k, resistor:R-EU_0207/15
- added R9: 30k, resistor:R-EU_0207/15
- added U$1: ISO6015, optocoupler:ISO6015
- added X2: 1751248, con-phoenix-350:1751248
- C1: value (none) -> 0.1u/250V; device capacitor-wima:C2,5-3 -> capacitor-wima:C5/5
- R1, R2: value (none) -> 360; device resistor:R-EU_0207/10 -> resistor:R-EU_0207/15
- R3: value (none) -> 220; device resistor:R-EU_0207/10 -> resistor:R-EU_0207/15
- R4: value (none) -> 10k; device resistor:R-EU_0207/10 -> resistor:R-EU_0207/15
- R5: value (none) -> 22; device resistor:R-EU_0207/10 -> resistor:R-EU_0309/12
- X1: value 87832-06 -> 1751316; device con-molex:87832-06 -> con-phoenix-350:1751316
Connections:
- removed net N$9: IC1.PB0, SL1.2
- new net N$15: OK1A.C, R8.1
- new net N$17: OK1A.E, X2-2.K
- new net N$19: F3.2
- new net N$21: OK1A.AC2, X1-6.K, X1-9.K
- net +5V: now also R3.2, R8.2, X1-7.K; no longer IC1.VCC, IC2.V+, R2.2, R5.2, SL1.6, X1.2
- net GND: now also R6.1, R9.2, U$1.C; no longer IC1.GND, IC2.GND, IC2.V-, R3.1, SL1.5, X1.6
- net N$1: now also OK1A.AC1, R7.2; no longer JP1.3
- net N$10: now also Q1.C, R3.1; no longer R1.1, SL1.1
- net N$11: now also Q1.E; no longer C1.1, IC2.+IN, R1.2
- net N$12: now also X1-8.K; no longer C1.2, IC2.-IN, R2.1, R3.2
- net N$13: now also Q1.B, R4.1; no longer IC2.ON, IC2.ON/STR
- net N$14: now also F3.1; no longer IC1.PB1, IC2.OUT, R4.1, R5.1
- net N$2: now also F1.2; no longer IC1.PA6, JP2.1, X1.4
- net N$3: now also F1.1; no longer IC1.PA5, X1.1
- net N$4: now also -.A2, C1.1, R1.2, R7.1, X1-4.K; no longer IC1.PB3, X1.5
- net N$5: now also -.A1, R2.1, R5.1, X1-5.K; no longer IC1.PA4, JP1.1, X1.3
- net N$6: now also R1.1, U$1.A2; no longer SL1.3
- net N$7: now also -.G, R2.2, U$1.A1; no longer JP2.3
- net N$8: now also C1.2, R5.2; no longer SL1.4
Other:
- note added: "L"
- note added: "N"
- note added: "in"
- note added: "triac-trig"
- note removed: "i2c-scl"
- note removed: "i2c-sda"
- note removed: "reset"
- note removed: "triac-trigger"
- moved on the sheet: C1, R1, R2, R3, R4, R5

Commit message: reg save
Parts:
- removed F1: FUSE 1A, fuse:FUSESH22,5
- removed F3: FUSE 16A, fuse:FUSESH22,5
- removed Q1: 2N2222A, transistor-npn:2N2222A
- removed R4, R6: 10k, resistor:R-EU_0207/15
- R3: value 220 -> 360
Connections:
- removed net N$10: Q1.C, R3.1
- removed net N$13: Q1.B, R4.1
- removed net N$14: F3.1
- removed net N$19: F3.2
- removed net N$2: F1.2
- removed net N$3: F1.1
- net +5V: no longer R3.2
- net GND: no longer R6.1
- net N$11: now also R3.2; no longer Q1.E
- net N$12: now also R3.1; no longer R4.2
Other:
- note removed: "in"
- moved on the sheet: R3
Changed lines of the file:
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@@
 <part name="R1" library="resistor" deviceset="R-EU_" device="0207/15" value="360"/>
 <part name="R2" library="resistor" deviceset="R-EU_" device="0207/15" value="360"/>
-<part name="R3" library="resistor" deviceset="R-EU_" device="0207/15" value="220"/>
-<part name="R4" library="resistor" deviceset="R-EU_" device="0207/15" value="10k"/>
-<part name="Q1" library="transistor-npn" deviceset="2N2222*" device="" technology="A"/>
-<part name="F3" library="fuse" deviceset="FUSE" device="SH22,5" value="FUSE 16A"/>
 <part name="FRAME1" library="frames" deviceset="A4L-LOC" device=""/>
 <part name="C1" library="capacitor-wima" deviceset="C" device="5/5" value="0.1u/250V"/>
@@
 <part name="SUPPLY3" library="supply2" deviceset="+5V" device=""/>
 <part name="R5" library="resistor" deviceset="R-EU_" device="0309/12" value="22"/>
-<part name="R6" library="resistor" deviceset="R-EU_" device="0207/15" value="10k"/>
 <part name="OK1" library="optocoupler" deviceset="TIL196" device=""/>
 <part name="R7" library="resistor" deviceset="R-EU_" device="0207/15" value="70k"/>
-<part name="F1" library="fuse" deviceset="FUSE" device="SH22,5" value="FUSE 1A"/>
 <part name="R8" library="resistor" deviceset="R-EU_" device="0207/15" value="1k"/>
 <part name="R9" library="resistor" deviceset="R-EU_" device="0207/15" value="30k"/>
 <part name="SUPPLY1" library="supply2" deviceset="GND" device=""/>
+<part name="R3" library="resistor" deviceset="R-EU_" device="0207/15" value="360"/>
 </parts>
 <sheets>
@@
 <text x="45.72" y="71.12" size="1.778" layer="91">N</text>
 <text x="35.56" y="60.96" size="1.778" layer="91">triac-trig</text>
-<text x="88.9" y="88.9" size="1.778" layer="91">in</text>
 </plain>
 <instances>
@@
 <instance part="R1" gate="G$1" x="-53.34" y="83.82" rot="R90"/>
 <instance part="R2" gate="G$1" x="-53.34" y="60.96" rot="R90"/>
-<instance part="R3" gate="G$1" x="-15.24" y="83.82"/>
-<instance part="R4" gate="G$1" x="0" y="58.42"/>
-<instance part="Q1" gate="G$1" x="-17.78" y="71.12" rot="MR0"/>
-<instance part="F3" gate="G$1" x="73.66" y="88.9"/>
 <instance part="FRAME1" gate="G$1" x="-116.84" y="-12.7"/>
 <instance part="C1" gate="G$1" x="30.48" y="88.9"/>
@@
 <instance part="SUPPLY3" gate="+5V" x="40.64" y="68.58"/>
 <instance part="R5" gate="G$1" x="30.48" y="81.28" rot="R90"/>
-<instance part="R6" gate="G$1" x="17.78" y="48.26" rot="R90"/>
 <instance part="OK1" gate="A" x="5.08" y="119.38"/>
 <instance part="R7" gate="G$1" x="-17.78" y="121.92"/>
-<instance part="F1" gate="G$1" x="73.66" y="73.66"/>
 <instance part="R8" gate="G$1" x="30.48" y="121.92"/>
 <instance part="R9" gate="G$1" x="30.48" y="111.76" rot="R270"/>
 <instance part="SUPPLY1" gate="GND" x="30.48" y="104.14"/>
+<instance part="R3" gate="G$1" x="-10.16" y="63.5" rot="R180"/>
 </instances>
 <busses>
@@
 <wire x1="-33.02" y1="66.04" x2="-27.94" y2="66.04" width="0.1524" layer="91"/>
 <wire x1="-27.94" y1="66.04" x2="-27.94" y2="43.18" width="0.1524" layer="91"/>
-<wire x1="-27.94" y1="43.18" x2="17.78" y2="43.18" width="0.1524" layer="91"/>
-<wire x1="17.78" y1="43.18" x2="27.94" y2="43.18" width="0.1524" layer="91"/>
-<wire x1="27.94" y1="43.18" x2="48.26" y2="43.18" width="0.1524" layer="91"/>
-<wire x1="50.8" y1="43.18" x2="48.26" y2="43.18" width="0.1524" layer="91"/>
+<wire x1="-27.94" y1="43.18" x2="27.94" y2="43.18" width="0.1524" layer="91"/>
+<wire x1="27.94" y1="43.18" x2="50.8" y2="43.18" width="0.1524" layer="91"/>
 <junction x="27.94" y="43.18"/>
-<junction x="17.78" y="43.18"/>
 <pinref part="U$1" gate="G$1" pin="C"/>
 <pinref part="SUPPLY2" gate="GND" pin="GND"/>
-<pinref part="R6" gate="G$1" pin="1"/>
 </segment>
 <segment>
@@
 </segment>
 </net>
-<net name="N$10" class="0">
-<segment>
-<wire x1="-20.32" y1="83.82" x2="-20.32" y2="76.2" width="0.1524" layer="91"/>
-<pinref part="R3" gate="G$1" pin="1"/>
-<pinref part="Q1" gate="G$1" pin="C"/>
-</segment>
-</net>
 <net name="N$11" class="0">
 <segment>
-<wire x1="-20.32" y1="66.04" x2="-25.4" y2="66.04" width="0.1524" layer="91"/>
-<wire x1="-25.4" y1="66.04" x2="-25.4" y2="76.2" width="0.1524" layer="91"/>
+<wire x1="-25.4" y1="63.5" x2="-25.4" y2="76.2" width="0.1524" layer="91"/>
 <wire x1="-25.4" y1="76.2" x2="-35.56" y2="76.2" width="0.1524" layer="91"/>
-<pinref part="Q1" gate="G$1" pin="E"/>
+<pinref part="R3" gate="G$1" pin="2"/>
+<wire x1="-15.24" y1="63.5" x2="-25.4" y2="63.5" width="0.1524" layer="91"/>
 </segment>
 </net>
 <net name="N$12" class="0">
 <segment>
-<wire x1="48.26" y1="58.42" x2="17.78" y2="58.42" width="0.1524" layer="91"/>
-<wire x1="17.78" y1="58.42" x2="5.08" y2="58.42" width="0.1524" layer="91"/>
-<wire x1="17.78" y1="58.42" x2="17.78" y2="50.8" width="0.1524" layer="91"/>
+<wire x1="48.26" y1="58.42" x2="15.24" y2="58.42" width="0.1524" layer="91"/>
 <pinref part="X1" gate="-8" pin="K"/>
-<pinref part="R4" gate="G$1" pin="2"/>
-</segment>
-</net>
-<net name="N$13" class="0">
-<segment>
-<wire x1="-5.08" y1="58.42" x2="-10.16" y2="58.42" width="0.1524" layer="91"/>
-<wire x1="-10.16" y1="58.42" x2="-10.16" y2="71.12" width="0.1524" layer="91"/>
-<wire x1="-10.16" y1="71.12" x2="-15.24" y2="71.12" width="0.1524" layer="91"/>
-<pinref part="R4" gate="G$1" pin="1"/>
-<pinref part="Q1" gate="G$1" pin="B"/>
-</segment>
-</net>
-<net name="N$14" class="0">
-<segment>
-<wire x1="63.5" y1="88.9" x2="68.58" y2="88.9" width="0.1524" layer="91"/>
-<wire x1="68.58" y1="88.9" x2="71.12" y2="88.9" width="0.1524" layer="91"/>
-<junction x="68.58" y="88.9"/>
-<pinref part="F3" gate="G$1" pin="1"/>
-</segment>
-</net>
-<net name="N$19" class="0">
-<segment>
-<wire x1="78.74" y1="88.9" x2="86.36" y2="88.9" width="0.1524" layer="91"/>
-<pinref part="F3" gate="G$1" pin="2"/>
+<wire x1="15.24" y1="58.42" x2="10.16" y2="58.42" width="0.1524" layer="91" curve="180"/>
+<wire x1="10.16" y1="58.42" x2="2.54" y2="58.42" width="0.1524" layer="91"/>
+<wire x1="2.54" y1="58.42" x2="2.54" y2="63.5" width="0.1524" layer="91"/>
+<pinref part="R3" gate="G$1" pin="1"/>
+<wire x1="2.54" y1="63.5" x2="-5.08" y2="63.5" width="0.1524" layer="91"/>
 </segment>
 </net>
 <net name="+5V" class="0">
 <segment>
+<pinref part="X1" gate="-7" pin="K"/>
 <wire x1="48.26" y1="66.04" x2="40.64" y2="66.04" width="0.1524" layer="91"/>
-<wire x1="40.64" y1="66.04" x2="7.62" y2="66.04" width="0.1524" layer="91"/>
+<pinref part="SUPPLY3" gate="+5V" pin="+5V"/>
+<wire x1="40.64" y1="66.04" x2="15.24" y2="66.04" width="0.1524" layer="91"/>
+<wire x1="15.24" y1="66.04" x2="10.16" y2="66.04" width="0.1524" layer="91" curve="180"/>
 <wire x1="7.62" y1="66.04" x2="7.62" y2="83.82" width="0.1524" layer="91"/>
 <wire x1="7.62" y1="83.82" x2="-5.08" y2="83.82" width="0.1524" layer="91"/>
-<junction x="40.64" y="66.04"/>
-<pinref part="X1" gate="-7" pin="K"/>
-<pinref part="R3" gate="G$1" pin="2"/>
-<pinref part="SUPPLY3" gate="+5V" pin="+5V"/>
-<wire x1="-5.08" y1="83.82" x2="-10.16" y2="83.82" width="0.1524" layer="91"/>
 <wire x1="-5.08" y1="83.82" x2="-5.08" y2="86.36" width="0.1524" layer="91"/>
 <wire x1="-5.08" y1="86.36" x2="-5.08" y2="91.44" width="0.1524" layer="91" curve="-180"/>
@@
 <pinref part="R8" gate="G$1" pin="2"/>
 <wire x1="38.1" y1="121.92" x2="35.56" y2="121.92" width="0.1524" layer="91"/>
+<wire x1="7.62" y1="66.04" x2="10.16" y2="66.04" width="0.1524" layer="91"/>
 </segment>
 </net>
@@
 </segment>
 </net>
-<net name="N$2" class="0">
-<segment>
-<wire x1="78.74" y1="73.66" x2="88.9" y2="73.66" width="0.1524" layer="91"/>
-<pinref part="F1" gate="G$1" pin="2"/>
-</segment>
-</net>
-<net name="N$3" class="0">
-<segment>
-<wire x1="68.58" y1="73.66" x2="63.5" y2="73.66" width="0.1524" layer="91"/>
-<pinref part="F1" gate="G$1" pin="1"/>
-</segment>
-</net>

Commit message: running application, designer 4.22, ide 1.12.1, debuggable
Parts:
- removed R9: 30k, resistor:R-EU_0207/15
- R8: value 1k -> 3k
Connections:
- removed net N$17: OK1A.E, X2-2.K
- net GND: now also OK1A.E; no longer R9.2
- net N$15: now also X2-2.K
Changed lines of the file:
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@@
 <part name="OK1" library="optocoupler" deviceset="TIL196" device=""/>
 <part name="R7" library="resistor" deviceset="R-EU_" device="0207/15" value="70k"/>
-<part name="R8" library="resistor" deviceset="R-EU_" device="0207/15" value="1k"/>
-<part name="R9" library="resistor" deviceset="R-EU_" device="0207/15" value="30k"/>
-<part name="SUPPLY1" library="supply2" deviceset="GND" device=""/>
+<part name="R8" library="resistor" deviceset="R-EU_" device="0207/15" value="3k"/>
 <part name="R3" library="resistor" deviceset="R-EU_" device="0207/15" value="360"/>
+<part name="SUPPLY4" library="supply2" deviceset="GND" device=""/>
 </parts>
 <sheets>
@@
 <instance part="R7" gate="G$1" x="-17.78" y="121.92"/>
 <instance part="R8" gate="G$1" x="30.48" y="121.92"/>
-<instance part="R9" gate="G$1" x="30.48" y="111.76" rot="R270"/>
-<instance part="SUPPLY1" gate="GND" x="30.48" y="104.14"/>
 <instance part="R3" gate="G$1" x="-10.16" y="63.5" rot="R180"/>
+<instance part="SUPPLY4" gate="GND" x="20.32" y="114.3"/>
 </instances>
 <busses>
@@
 </segment>
 <segment>
-<pinref part="R9" gate="G$1" pin="2"/>
-<pinref part="SUPPLY1" gate="GND" pin="GND"/>
+<pinref part="OK1" gate="A" pin="E"/>
+<pinref part="SUPPLY4" gate="GND" pin="GND"/>
+<wire x1="17.78" y1="116.84" x2="20.32" y2="116.84" width="0.1524" layer="91"/>
 </segment>
 </net>
@@
 <pinref part="R8" gate="G$1" pin="1"/>
 <wire x1="17.78" y1="121.92" x2="25.4" y2="121.92" width="0.1524" layer="91"/>
-</segment>
-</net>
-<net name="N$17" class="0">
-<segment>
-<pinref part="OK1" gate="A" pin="E"/>
-<wire x1="17.78" y1="116.84" x2="129.54" y2="116.84" width="0.1524" layer="91"/>
+<wire x1="25.4" y1="121.92" x2="25.4" y2="116.84" width="0.1524" layer="91"/>
 <wire x1="129.54" y1="116.84" x2="129.54" y2="25.4" width="0.1524" layer="91"/>
 <wire x1="129.54" y1="25.4" x2="43.18" y2="25.4" width="0.1524" layer="91"/>
@@
 <pinref part="X2" gate="-2" pin="K"/>
 <wire x1="43.18" y1="35.56" x2="48.26" y2="35.56" width="0.1524" layer="91"/>
-</segment>
-</net>
+<wire x1="25.4" y1="116.84" x2="129.54" y2="116.84" width="0.1524" layer="91"/>
+</segment>
+</net>

Commit message: reg save, runs as never before :-), EAGLE CHANGES
Parts:
- added C2: 0.05U, resistor:C-EU025-040X050
- added R4: 100, resistor:R-EU_0207/15
- R1: value 360 -> 300
- R2: value 360 -> 470
Connections:
- removed net N$12: R3.1, X1-8.K
- new net N$10: -.A2, C1.1, R2.1, R7.1, X1-4.K
- new net N$2: C2.2, R4.2, R5.1, X1-5.K
- new net N$3: R3.1
- new net N$9: -.A1
- net GND: now also U$1.A1; no longer U$1.C
- net N$11: now also R4.1, U$1.C; no longer R3.2
- net N$4: now also -.G; no longer -.A2, C1.1, R1.2, R7.1, X1-4.K
- net N$5: now also C2.1, R1.2, R2.2; no longer -.A1, R2.1, R5.1, X1-5.K
- net N$6: now also R3.2, X1-8.K; no longer R1.1, U$1.A2
- net N$7: now also R1.1, U$1.A; no longer -.G, R2.2, U$1.A1
Other:
- note added: "====="
- note added: "MOC3021"
- moved on the sheet: -, R1, R2, R3, U$1

Commit message: reg save, minor changes
Parts:
- R3: value 360 -> 220
Connections:
- removed net N$11: R4.1, U$1.C
- removed net N$3: R3.1
- new net N$12: R4.1, U$1.A1
- new net N$13: R3.1, U$1.A
- net GND: now also U$1.C; no longer U$1.A1
- net N$7: now also U$1.A2; no longer U$1.A
Changed lines of the file:
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@@
 <part name="R7" library="resistor" deviceset="R-EU_" device="0207/15" value="70k"/>
 <part name="R8" library="resistor" deviceset="R-EU_" device="0207/15" value="3k"/>
-<part name="R3" library="resistor" deviceset="R-EU_" device="0207/15" value="360"/>
+<part name="R3" library="resistor" deviceset="R-EU_" device="0207/15" value="220"/>
 <part name="SUPPLY4" library="supply2" deviceset="GND" device=""/>
 <part name="SUPPLY1" library="supply2" deviceset="GND" device=""/>
@@
 <text x="45.72" y="71.12" size="1.778" layer="91">N</text>
 <text x="35.56" y="60.96" size="1.778" layer="91">triac-trig</text>
-<text x="-86.36" y="58.42" size="1.778" layer="91">MOC3021</text>
-<text x="-86.36" y="60.96" size="1.778" layer="91">=====</text>
+<text x="-93.98" y="58.42" size="1.778" layer="91">MOC3021</text>
+<text x="-93.98" y="60.96" size="1.778" layer="91">=====</text>
 <text x="-88.9" y="60.96" size="1.778" layer="91">=====</text>
 </plain>
@@
 <instance part="X2" gate="-1" x="50.8" y="43.18"/>
 <instance part="X2" gate="-2" x="50.8" y="35.56"/>
-<instance part="U$1" gate="G$1" x="-86.36" y="71.12" rot="MR0"/>
+<instance part="U$1" gate="G$1" x="-86.36" y="71.12"/>
 <instance part="R1" gate="G$1" x="-68.58" y="88.9"/>
 <instance part="R2" gate="G$1" x="-48.26" y="88.9" rot="MR0"/>
@@
 <instance part="R3" gate="G$1" x="-104.14" y="76.2" rot="R180"/>
 <instance part="SUPPLY4" gate="GND" x="20.32" y="114.3"/>
-<instance part="SUPPLY1" gate="GND" x="-96.52" y="55.88"/>
+<instance part="SUPPLY1" gate="GND" x="-99.06" y="55.88"/>
 <instance part="C2" gate="G$1" x="-60.96" y="66.04"/>
 <instance part="R4" gate="G$1" x="-40.64" y="60.96" rot="R270"/>
@@
 </segment>
 <segment>
-<pinref part="U$1" gate="G$1" pin="A1"/>
-<wire x1="-96.52" y1="66.04" x2="-96.52" y2="58.42" width="0.1524" layer="91"/>
+<pinref part="U$1" gate="G$1" pin="C"/>
+<wire x1="-96.52" y1="66.04" x2="-99.06" y2="66.04" width="0.1524" layer="91"/>
 <pinref part="SUPPLY1" gate="GND" pin="GND"/>
+<wire x1="-99.06" y1="66.04" x2="-99.06" y2="58.42" width="0.1524" layer="91"/>
 </segment>
 </net>
@@
 </segment>
 </net>
-<net name="N$3" class="0">
-<segment>
-<pinref part="R3" gate="G$1" pin="1"/>
-<wire x1="-99.06" y1="76.2" x2="-93.98" y2="76.2" width="0.1524" layer="91"/>
-</segment>
-</net>
 <net name="N$6" class="0">
 <segment>
@@
 <net name="N$7" class="0">
 <segment>
-<pinref part="U$1" gate="G$1" pin="A"/>
+<pinref part="U$1" gate="G$1" pin="A2"/>
+<wire x1="-76.2" y1="76.2" x2="-76.2" y2="88.9" width="0.1524" layer="91"/>
 <pinref part="R1" gate="G$1" pin="1"/>
-<wire x1="-76.2" y1="76.2" x2="-73.66" y2="76.2" width="0.1524" layer="91"/>
-<wire x1="-73.66" y1="76.2" x2="-73.66" y2="88.9" width="0.1524" layer="91"/>
+<wire x1="-76.2" y1="88.9" x2="-73.66" y2="88.9" width="0.1524" layer="91"/>
 </segment>
 </net>
@@
 </segment>
 </net>
-<net name="N$11" class="0">
-<segment>
-<pinref part="U$1" gate="G$1" pin="C"/>
-<wire x1="-76.2" y1="66.04" x2="-76.2" y2="71.12" width="0.1524" layer="91"/>
-<wire x1="-76.2" y1="71.12" x2="-63.5" y2="71.12" width="0.1524" layer="91"/>
+<net name="N$12" class="0">
+<segment>
+<pinref part="U$1" gate="G$1" pin="A1"/>
+<wire x1="-76.2" y1="66.04" x2="-68.58" y2="66.04" width="0.1524" layer="91"/>
+<wire x1="-68.58" y1="66.04" x2="-68.58" y2="71.12" width="0.1524" layer="91"/>
 <wire x1="-63.5" y1="71.12" x2="-58.42" y2="71.12" width="0.1524" layer="91" curve="-180"/>
 <wire x1="-58.42" y1="71.12" x2="-40.64" y2="71.12" width="0.1524" layer="91"/>
 <pinref part="R4" gate="G$1" pin="1"/>
 <wire x1="-40.64" y1="71.12" x2="-40.64" y2="66.04" width="0.1524" layer="91"/>
-</segment>
-</net>
+<wire x1="-68.58" y1="71.12" x2="-66.04" y2="71.12" width="0.1524" layer="91"/>
+<wire x1="-63.5" y1="71.12" x2="-66.04" y2="71.12" width="0.1524" layer="91"/>
+</segment>
+</net>
+<net name="N$13" class="0">
+<segment>
+<pinref part="U$1" gate="G$1" pin="A"/>
+<pinref part="R3" gate="G$1" pin="1"/>
+<wire x1="-99.06" y1="76.2" x2="-96.52" y2="76.2" width="0.1524" layer="91"/>
+</segment>
+</net>

Commit message: reg save
Parts:
- removed R4: 100, resistor:R-EU_0207/15
Connections:
- net N$12: no longer R4.1
- net N$2: no longer R4.2
Changed lines of the file:
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@@
 <part name="SUPPLY1" library="supply2" deviceset="GND" device=""/>
 <part name="C2" library="resistor" deviceset="C-EU" device="025-040X050" value="0.05U"/>
-<part name="R4" library="resistor" deviceset="R-EU_" device="0207/15" value="100"/>
 </parts>
 <sheets>
@@
 <instance part="SUPPLY1" gate="GND" x="-99.06" y="55.88"/>
 <instance part="C2" gate="G$1" x="-60.96" y="66.04"/>
-<instance part="R4" gate="G$1" x="-40.64" y="60.96" rot="R270"/>
 </instances>
 <busses>
@@
 <pinref part="C2" gate="G$1" pin="2"/>
 <wire x1="-60.96" y1="60.96" x2="-60.96" y2="50.8" width="0.1524" layer="91"/>
-<wire x1="-60.96" y1="50.8" x2="-40.64" y2="50.8" width="0.1524" layer="91"/>
-<pinref part="R4" gate="G$1" pin="2"/>
-<wire x1="-40.64" y1="50.8" x2="12.7" y2="50.8" width="0.1524" layer="91"/>
-<wire x1="-40.64" y1="55.88" x2="-40.64" y2="50.8" width="0.1524" layer="91"/>
+<wire x1="-60.96" y1="50.8" x2="12.7" y2="50.8" width="0.1524" layer="91"/>
 </segment>
 </net>
@@
 <wire x1="-63.5" y1="71.12" x2="-58.42" y2="71.12" width="0.1524" layer="91" curve="-180"/>
 <wire x1="-58.42" y1="71.12" x2="-40.64" y2="71.12" width="0.1524" layer="91"/>
-<pinref part="R4" gate="G$1" pin="1"/>
-<wire x1="-40.64" y1="71.12" x2="-40.64" y2="66.04" width="0.1524" layer="91"/>
-<wire x1="-68.58" y1="71.12" x2="-66.04" y2="71.12" width="0.1524" layer="91"/>
-<wire x1="-63.5" y1="71.12" x2="-66.04" y2="71.12" width="0.1524" layer="91"/>
-</segment>
-</net>
+<wire x1="-63.5" y1="71.12" x2="-68.58" y2="71.12" width="0.1524" layer="91"/>
+</segment>
+</net>
