File: eagle/joesTriac/joesTriac-2nd/cpuConnectionBoard.sch (EAGLE design)
At the start: 12 parts, among them IC1 24C01CP, J1 CN11, J2 CN9, J3 CN13, J4 CN14, Q1 2N4403, Q2 2N4401

Commit message: reg save, eclipse changes
Parts:
- added IC2: LM311N, linear:LM311N
- added J5: CN9, con-omron:XF2E-1015-1
- added R5, R7: 2.2k, resistor:R-EU_0309/12
- added R6: 2k, resistor:R-TRIMM64P
- added R8: 330k, resistor:R-EU_0309/12
Connections:
- new net N$10: IC2.-IN
- new net N$11: R5.2, R6.A
- new net N$12: IC2.+IN, R6.S, R8.1
- new net N$13: J2-5.MS
- new net N$14: J2-1.MSV
- new net N$15: J2-2.MS
- new net N$16: IC2.ON, IC2.V+
- new net N$17: IC2.ON/STR, R7.1
- new net N$18: J3-1.MSV
- new net N$7: IC2.OUT, R8.2
- new net N$9: J5-8.MS
- net +5V: now also R6.E, R7.2
- net GND: now also IC2.V-, R5.1
- net N$8: now also J5-5.MS; no longer J2-9.MS
Other:
- note added: "PA12"
- note added: "VoltageZeroPass"
- note added: "connector to boards"
- moved on the sheet: J3-1, J3-2, J3-3, J3-4, J3-5, J3-6, J3-7, J3-8, J4-1, J4-2, J4-3, J4-4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
Changed lines of the file:
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@@
 <part name="SUPPLY7" library="supply2" deviceset="GND" device=""/>
 <part name="R4" library="resistor" deviceset="R-EU_" device="0309/12" value="47k"/>
+<part name="IC2" library="linear" deviceset="LM311" device="N"/>
+<part name="J5" library="con-omron" deviceset="XF2*-10?" device="15-1" technology="E" value="CN9"/>
+<part name="R5" library="resistor" deviceset="R-EU_" device="0309/12" value="2.2k"/>
+<part name="SUPPLY8" library="supply2" deviceset="GND" device=""/>
+<part name="R6" library="resistor" deviceset="R-TRIMM" device="64P" value="2k"/>
+<part name="SUPPLY9" library="supply2" deviceset="+5V" device=""/>
+<part name="SUPPLY10" library="supply2" deviceset="+5V" device=""/>
+<part name="SUPPLY11" library="supply2" deviceset="GND" device=""/>
+<part name="R7" library="resistor" deviceset="R-EU_" device="0309/12" value="2.2k"/>
+<part name="R8" library="resistor" deviceset="R-EU_" device="0309/12" value="330k"/>
 </parts>
 <sheets>
@@
 <text x="88.9" y="0" size="1.778" layer="91">out</text>
 <text x="-15.24" y="48.26" size="1.778" layer="91">PH6</text>
-<text x="124.46" y="38.1" size="1.778" layer="91">triac trigger</text>
+<text x="124.46" y="46.482" size="1.778" layer="91">triac trigger</text>
+<text x="162.56" y="60.96" size="1.778" layer="91">connector to boards</text>
+<text x="139.7" y="31.242" size="1.778" layer="91">VoltageZeroPass</text>
+<text x="-22.86" y="3.302" size="1.778" layer="91">VoltageZeroPass</text>
+<text x="-15.24" y="40.64" size="1.778" layer="91">PA12</text>
+<text x="147.32" y="-6.858" size="1.778" layer="91">PA12</text>
+<text x="152.4" y="3.556" size="1.778" layer="91">PB8</text>
+<text x="144.78" y="1.016" size="1.778" layer="91">PB9</text>
+<text x="152.4" y="-26.67" size="1.778" layer="91">PH6</text>
 </plain>
 <instances>
@@
 <instance part="J2" gate="-9" x="160.02" y="-17.78"/>
 <instance part="J2" gate="-10" x="160.02" y="-20.32"/>
-<instance part="J3" gate="-1" x="160.02" y="-43.18"/>
-<instance part="J3" gate="-2" x="160.02" y="-45.72"/>
-<instance part="J3" gate="-3" x="160.02" y="-48.26"/>
-<instance part="J3" gate="-4" x="160.02" y="-50.8"/>
-<instance part="J3" gate="-5" x="160.02" y="-53.34"/>
-<instance part="J3" gate="-6" x="160.02" y="-55.88"/>
-<instance part="J3" gate="-7" x="160.02" y="-58.42"/>
-<instance part="J3" gate="-8" x="160.02" y="-60.96"/>
-<instance part="J4" gate="-1" x="78.74" y="-30.48"/>
-<instance part="J4" gate="-2" x="78.74" y="-33.02"/>
-<instance part="J4" gate="-3" x="78.74" y="-35.56"/>
-<instance part="J4" gate="-4" x="78.74" y="-38.1"/>
-<instance part="J4" gate="-5" x="78.74" y="-40.64"/>
-<instance part="J4" gate="-6" x="78.74" y="-43.18"/>
+<instance part="J3" gate="-1" x="160.02" y="-27.94"/>
+<instance part="J3" gate="-2" x="160.02" y="-30.48"/>
+<instance part="J3" gate="-3" x="160.02" y="-33.02"/>
+<instance part="J3" gate="-4" x="160.02" y="-35.56"/>
+<instance part="J3" gate="-5" x="160.02" y="-38.1"/>
+<instance part="J3" gate="-6" x="160.02" y="-40.64"/>
+<instance part="J3" gate="-7" x="160.02" y="-43.18"/>
+<instance part="J3" gate="-8" x="160.02" y="-45.72"/>
+<instance part="J4" gate="-1" x="78.74" y="-25.4"/>
+<instance part="J4" gate="-2" x="78.74" y="-27.94"/>
+<instance part="J4" gate="-3" x="78.74" y="-30.48"/>
+<instance part="J4" gate="-4" x="78.74" y="-33.02"/>
+<instance part="J4" gate="-5" x="78.74" y="-35.56"/>
+<instance part="J4" gate="-6" x="78.74" y="-38.1"/>
 <instance part="Q1" gate="A" x="114.3" y="58.42"/>
 <instance part="R1" gate="G$1" x="73.66" y="30.48"/>
@@
 <instance part="SUPPLY7" gate="GND" x="104.14" y="15.24"/>
 <instance part="R4" gate="G$1" x="116.84" y="27.94" rot="R90"/>
+<instance part="IC2" gate="A" x="5.08" y="5.08"/>
+<instance part="J5" gate="-1" x="162.56" y="55.88"/>
+<instance part="J5" gate="-2" x="162.56" y="53.34"/>
+<instance part="J5" gate="-3" x="162.56" y="50.8"/>
+<instance part="J5" gate="-4" x="162.56" y="48.26"/>
+<instance part="J5" gate="-5" x="162.56" y="45.72"/>
+<instance part="J5" gate="-6" x="162.56" y="43.18"/>
+<instance part="J5" gate="-7" x="162.56" y="40.64"/>
+<instance part="J5" gate="-8" x="162.56" y="38.1"/>
+<instance part="R5" gate="G$1" x="-27.94" y="-2.54" rot="R90"/>
+<instance part="SUPPLY8" gate="GND" x="-27.94" y="-10.16"/>
+<instance part="R6" gate="G$1" x="-27.94" y="10.16"/>
+<instance part="SUPPLY9" gate="+5V" x="-27.94" y="17.78"/>
+<instance part="SUPPLY10" gate="+5V" x="12.7" y="20.32"/>
+<instance part="SUPPLY11" gate="GND" x="7.62" y="-5.08"/>
+<instance part="R7" gate="G$1" x="12.7" y="12.7" rot="R90"/>
+<instance part="R8" gate="G$1" x="-5.08" y="17.78" rot="R90"/>
 </instances>
 <busses>
@@
 <wire x1="76.2" y1="-5.08" x2="55.88" y2="-5.08" width="0.1524" layer="91"/>
 <pinref part="SUPPLY4" gate="+5V" pin="+5V"/>
+</segment>
+<segment>
+<pinref part="R6" gate="G$1" pin="E"/>
+<pinref part="SUPPLY9" gate="+5V" pin="+5V"/>
+</segment>
+<segment>
+<pinref part="SUPPLY10" gate="+5V" pin="+5V"/>
+<pinref part="R7" gate="G$1" pin="2"/>
 </segment>
 </net>
@@
 <pinref part="SUPPLY5" gate="GND" pin="GND"/>
 <junction x="58.42" y="-10.16"/>
-<wire x1="58.42" y1="-10.16" x2="25.4" y2="-10.16" width="0.1524" layer="91"/>
-<wire x1="25.4" y1="-10.16" x2="25.4" y2="17.78" width="0.1524" layer="91"/>
-<wire x1="25.4" y1="17.78" x2="83.82" y2="17.78" width="0.1524" layer="91"/>
+<wire x1="58.42" y1="-10.16" x2="50.8" y2="-10.16" width="0.1524" layer="91"/>
+<wire x1="50.8" y1="-10.16" x2="50.8" y2="17.78" width="0.1524" layer="91"/>
+<wire x1="50.8" y1="17.78" x2="83.82" y2="17.78" width="0.1524" layer="91"/>
 <pinref part="Q2" gate="G$1" pin="E"/>
 <wire x1="83.82" y1="17.78" x2="104.14" y2="17.78" width="0.1524" layer="91"/>
@@
 <pinref part="SUPPLY6" gate="GND" pin="GND"/>
 </segment>
+<segment>
+<pinref part="R5" gate="G$1" pin="1"/>
+<pinref part="SUPPLY8" gate="GND" pin="GND"/>
+</segment>
+<segment>
+<pinref part="IC2" gate="A" pin="V-"/>
+<wire x1="2.54" y1="-2.54" x2="7.62" y2="-2.54" width="0.1524" layer="91"/>
+<pinref part="SUPPLY11" gate="GND" pin="GND"/>
+</segment>
 </net>
 <net name="N$2" class="0">
@@
 <segment>
 <pinref part="Q1" gate="A" pin="C"/>
-<wire x1="116.84" y1="53.34" x2="116.84" y2="38.1" width="0.1524" layer="91"/>
 <pinref part="R4" gate="G$1" pin="2"/>
-<wire x1="116.84" y1="38.1" x2="116.84" y2="33.02" width="0.1524" layer="91"/>
-<wire x1="116.84" y1="38.1" x2="121.92" y2="38.1" width="0.1524" layer="91"/>
-<wire x1="121.92" y1="38.1" x2="121.92" y2="-17.78" width="0.1524" layer="91"/>
-<pinref part="J2" gate="-9" pin="MS"/>
-<wire x1="121.92" y1="-17.78" x2="157.48" y2="-17.78" width="0.1524" layer="91"/>
-</segment>
-</net>
+<wire x1="116.84" y1="53.34" x2="116.84" y2="45.72" width="0.1524" layer="91"/>
+<pinref part="J5" gate="-5" pin="MS"/>
+<wire x1="116.84" y1="45.72" x2="116.84" y2="33.02" width="0.1524" layer="91"/>
+<wire x1="160.02" y1="45.72" x2="116.84" y2="45.72" width="0.1524" layer="91"/>
+</segment>
+</net>
+<net name="N$7" class="0">
+<segment>
+<wire x1="-17.78" y1="40.64" x2="-12.7" y2="40.64" width="0.1524" layer="91"/>
+<wire x1="-12.7" y1="40.64" x2="-12.7" y2="27.94" width="0.1524" layer="91"/>
+<pinref part="IC2" gate="A" pin="OUT"/>
+<wire x1="12.7" y1="5.08" x2="20.32" y2="5.08" width="0.1524" layer="91"/>
+<wire x1="20.32" y1="5.08" x2="20.32" y2="27.94" width="0.1524" layer="91"/>
+<wire x1="20.32" y1="27.94" x2="-5.08" y2="27.94" width="0.1524" layer="91"/>
+<pinref part="R8" gate="G$1" pin="2"/>
+<wire x1="-5.08" y1="27.94" x2="-12.7" y2="27.94" width="0.1524" layer="91"/>
+<wire x1="-5.08" y1="27.94" x2="-5.08" y2="22.86" width="0.1524" layer="91"/>
+</segment>
+</net>
+<net name="N$9" class="0">
+<segment>
+<pinref part="J5" gate="-8" pin="MS"/>
+<wire x1="160.02" y1="38.1" x2="160.02" y2="30.48" width="0.1524" layer="91"/>
+<wire x1="160.02" y1="30.48" x2="142.24" y2="30.48" width="0.1524" layer="91"/>
+</segment>
+</net>
+<net name="N$10" class="0">
+<segment>
+<pinref part="IC2" gate="A" pin="-IN"/>
+<wire x1="-2.54" y1="2.54" x2="-22.86" y2="2.54" width="0.1524" layer="91"/>
+</segment>
+</net>
+<net name="N$11" class="0">
+<segment>
+<pinref part="R6" gate="G$1" pin="A"/>
+<pinref part="R5" gate="G$1" pin="2"/>
+<wire x1="-27.94" y1="5.08" x2="-27.94" y2="2.54" width="0.1524" layer="91"/>
+</segment>
+</net>
+<net name="N$12" class="0">
+<segment>
+<pinref part="R6" gate="G$1" pin="S"/>
+<wire x1="-22.86" y1="10.16" x2="-22.86" y2="7.62" width="0.1524" layer="91"/>
+<pinref part="IC2" gate="A" pin="+IN"/>
+<wire x1="-22.86" y1="7.62" x2="-5.08" y2="7.62" width="0.1524" layer="91"/>
+<pinref part="R8" gate="G$1" pin="1"/>
+<wire x1="-5.08" y1="7.62" x2="-2.54" y2="7.62" width="0.1524" layer="91"/>
+<wire x1="-5.08" y1="12.7" x2="-5.08" y2="7.62" width="0.1524" layer="91"/>
+</segment>
+</net>
+<net name="N$13" class="0">
+<segment>
+<pinref part="J2" gate="-5" pin="MS"/>
+<wire x1="157.48" y1="-7.62" x2="147.32" y2="-7.62" width="0.1524" layer="91"/>
+</segment>
+</net>
+<net name="N$14" class="0">
+<segment>
+<pinref part="J2" gate="-1" pin="MSV"/>
+<wire x1="157.48" y1="2.54" x2="152.4" y2="2.54" width="0.1524" layer="91"/>
+</segment>
+</net>
+<net name="N$15" class="0">
+<segment>
+<pinref part="J2" gate="-2" pin="MS"/>
+<wire x1="157.48" y1="0" x2="144.78" y2="0" width="0.1524" layer="91"/>
+</segment>
+</net>
+<net name="N$16" class="0">
+<segment>
+<pinref part="IC2" gate="A" pin="V+"/>
+<pinref part="IC2" gate="A" pin="ON"/>
+<wire x1="2.54" y1="12.7" x2="5.08" y2="12.7" width="0.1524" layer="91"/>
+</segment>
+</net>
+<net name="N$17" class="0">
+<segment>
+<pinref part="IC2" gate="A" pin="ON/STR"/>
+<pinref part="R7" gate="G$1" pin="1"/>
+</segment>
+</net>
+<net name="N$18" class="0">
+<segment>
+<pinref part="J3" gate="-1" pin="MSV"/>
+<wire x1="157.48" y1="-27.94" x2="152.4" y2="-27.94" width="0.1524" layer="91"/>
+</segment>
+</net>

Commit message: reg save, working on exti
Parts:
- added C2, C3: 10uF, resistor:C-EU050-030X075
- added L1: SMCC12, inductors:SMCC12
Connections:
- new net N$19: C3.1, L1.1
- new net N$20: C2.1, L1.2
- net GND: now also C2.2, C3.2
Changed lines of the file:
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@@
 <part name="R7" library="resistor" deviceset="R-EU_" device="0309/12" value="2.2k"/>
 <part name="R8" library="resistor" deviceset="R-EU_" device="0309/12" value="330k"/>
+<part name="L1" library="inductors" deviceset="SMCC12" device=""/>
+<part name="C2" library="resistor" deviceset="C-EU" device="050-030X075" value="10uF"/>
+<part name="C3" library="resistor" deviceset="C-EU" device="050-030X075" value="10uF"/>
+<part name="SUPPLY12" library="supply2" deviceset="GND" device=""/>
 </parts>
 <sheets>
@@
 <instance part="R7" gate="G$1" x="12.7" y="12.7" rot="R90"/>
 <instance part="R8" gate="G$1" x="-5.08" y="17.78" rot="R90"/>
+<instance part="L1" gate="1" x="-5.08" y="-17.78"/>
+<instance part="C2" gate="G$1" x="5.08" y="-22.86"/>
+<instance part="C3" gate="G$1" x="-15.24" y="-22.86"/>
+<instance part="SUPPLY12" gate="GND" x="12.7" y="-35.56"/>
 </instances>
 <busses>
@@
 <pinref part="SUPPLY11" gate="GND" pin="GND"/>
 </segment>
+<segment>
+<wire x1="-25.4" y1="-33.02" x2="-15.24" y2="-33.02" width="0.1524" layer="91" style="shortdash"/>
+<pinref part="SUPPLY12" gate="GND" pin="GND"/>
+<wire x1="-15.24" y1="-33.02" x2="5.08" y2="-33.02" width="0.1524" layer="91" style="shortdash"/>
+<wire x1="5.08" y1="-33.02" x2="12.7" y2="-33.02" width="0.1524" layer="91" style="shortdash"/>
+<wire x1="12.7" y1="-33.02" x2="17.78" y2="-33.02" width="0.1524" layer="91" style="shortdash"/>
+<junction x="12.7" y="-33.02"/>
+<pinref part="C3" gate="G$1" pin="2"/>
+<wire x1="-15.24" y1="-27.94" x2="-15.24" y2="-33.02" width="0.1524" layer="91" style="shortdash"/>
+<pinref part="C2" gate="G$1" pin="2"/>
+<wire x1="5.08" y1="-27.94" x2="5.08" y2="-33.02" width="0.1524" layer="91" style="shortdash"/>
+</segment>
 </net>
 <net name="N$2" class="0">
@@
 <pinref part="IC2" gate="A" pin="-IN"/>
 <wire x1="-2.54" y1="2.54" x2="-22.86" y2="2.54" width="0.1524" layer="91"/>
+<wire x1="-22.86" y1="2.54" x2="-22.86" y2="-17.78" width="0.1524" layer="91"/>
+<wire x1="-22.86" y1="-17.78" x2="-20.32" y2="-17.78" width="0.1524" layer="91"/>
 </segment>
 </net>
@@
 </segment>
 </net>
+<net name="N$19" class="0">
+<segment>
+<pinref part="L1" gate="1" pin="1"/>
+<wire x1="-17.78" y1="-17.78" x2="-15.24" y2="-17.78" width="0.1524" layer="91" style="shortdash"/>
+<wire x1="-12.7" y1="-17.78" x2="-15.24" y2="-17.78" width="0.1524" layer="91" style="shortdash"/>
+<pinref part="C3" gate="G$1" pin="1"/>
+<wire x1="-15.24" y1="-17.78" x2="-15.24" y2="-20.32" width="0.1524" layer="91" style="shortdash"/>
+</segment>
+</net>
+<net name="N$20" class="0">
+<segment>
+<pinref part="L1" gate="1" pin="2"/>
+<wire x1="2.54" y1="-17.78" x2="5.08" y2="-17.78" width="0.1524" layer="91" style="shortdash"/>
+<wire x1="12.7" y1="-17.78" x2="5.08" y2="-17.78" width="0.1524" layer="91" style="shortdash"/>
+<pinref part="C2" gate="G$1" pin="1"/>
+<wire x1="5.08" y1="-17.78" x2="5.08" y2="-20.32" width="0.1524" layer="91" style="shortdash"/>
+</segment>
+</net>

Commit message: reg save, working on exti spikes
Parts:
- added C4: 47nF, resistor:C-EU050-030X075
- added C5: 22nF, resistor:C-EU050-030X075
- added L2: SMCC12, inductors:SMCC12
- C2: value 10uF -> 47nF
- C3: value 10uF -> 22nF
Connections:
- new net N$34: C4.1, L2.2
- new net N$35: C5.1, L2.1
- net GND: now also C4.2, C5.2
- net N$10: now also C3.1
- net N$19: now also J4-1.MSV; no longer C3.1, L1.1
Other:
- note added: "PA6"
- note added: "adc"
Changed lines of the file:
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@@
 <layer number="98" name="Guide" color="6" fill="1" visible="yes" active="yes"/>
 <layer number="99" name="SpiceOrder" color="5" fill="1" visible="yes" active="yes"/>
+<layer number="101" name="Hidden" color="15" fill="1" visible="yes" active="yes"/>
+<layer number="102" name="Changes" color="12" fill="1" visible="yes" active="yes"/>
 </layers>
 <schematic xreflabel="%F%N/%S.%C%R" xrefpart="/%S.%C%R">
@@
 <part name="R8" library="resistor" deviceset="R-EU_" device="0309/12" value="330k"/>
 <part name="L1" library="inductors" deviceset="SMCC12" device=""/>
-<part name="C2" library="resistor" deviceset="C-EU" device="050-030X075" value="10uF"/>
-<part name="C3" library="resistor" deviceset="C-EU" device="050-030X075" value="10uF"/>
+<part name="C2" library="resistor" deviceset="C-EU" device="050-030X075" value="47nF"/>
+<part name="C3" library="resistor" deviceset="C-EU" device="050-030X075" value="22nF"/>
 <part name="SUPPLY12" library="supply2" deviceset="GND" device=""/>
+<part name="L2" library="inductors" deviceset="SMCC12" device=""/>
+<part name="C4" library="resistor" deviceset="C-EU" device="050-030X075" value="47nF"/>
+<part name="C5" library="resistor" deviceset="C-EU" device="050-030X075" value="22nF"/>
+<part name="SUPPLY33" library="supply2" deviceset="GND" device=""/>
 </parts>
 <sheets>
@@
 <text x="144.78" y="1.016" size="1.778" layer="91">PB9</text>
 <text x="152.4" y="-26.67" size="1.778" layer="91">PH6</text>
+<text x="5.08" y="-17.018" size="1.778" layer="91">VoltageZeroPass</text>
+<text x="-55.88" y="43.18" size="1.778" layer="91">PA6</text>
+<text x="-50.8" y="19.05" size="1.778" layer="91">adc</text>
+<text x="66.04" y="-22.86" size="1.778" layer="91">adc</text>
 </plain>
 <instances>
@@
 <instance part="J5" gate="-8" x="162.56" y="38.1"/>
 <instance part="R5" gate="G$1" x="-27.94" y="-2.54" rot="R90"/>
-<instance part="SUPPLY8" gate="GND" x="-27.94" y="-10.16"/>
+<instance part="SUPPLY8" gate="GND" x="-27.94" y="-12.7"/>
 <instance part="R6" gate="G$1" x="-27.94" y="10.16"/>
 <instance part="SUPPLY9" gate="+5V" x="-27.94" y="17.78"/>
@@
 <instance part="C2" gate="G$1" x="5.08" y="-22.86"/>
 <instance part="C3" gate="G$1" x="-15.24" y="-22.86"/>
-<instance part="SUPPLY12" gate="GND" x="12.7" y="-35.56"/>
+<instance part="SUPPLY12" gate="GND" x="12.7" y="-33.02"/>
+<instance part="L2" gate="1" x="-66.04" y="17.78"/>
+<instance part="C4" gate="G$1" x="-55.88" y="12.7"/>
+<instance part="C5" gate="G$1" x="-76.2" y="12.7"/>
+<instance part="SUPPLY33" gate="GND" x="-48.26" y="2.54"/>
 </instances>
 <busses>
@@
 <pinref part="R5" gate="G$1" pin="1"/>
 <pinref part="SUPPLY8" gate="GND" pin="GND"/>
+<wire x1="-27.94" y1="-10.16" x2="-27.94" y2="-7.62" width="0.1524" layer="91"/>
 </segment>
 <segment>
@@
 </segment>
 <segment>
-<wire x1="-25.4" y1="-33.02" x2="-15.24" y2="-33.02" width="0.1524" layer="91" style="shortdash"/>
 <pinref part="SUPPLY12" gate="GND" pin="GND"/>
-<wire x1="-15.24" y1="-33.02" x2="5.08" y2="-33.02" width="0.1524" layer="91" style="shortdash"/>
-<wire x1="5.08" y1="-33.02" x2="12.7" y2="-33.02" width="0.1524" layer="91" style="shortdash"/>
-<wire x1="12.7" y1="-33.02" x2="17.78" y2="-33.02" width="0.1524" layer="91" style="shortdash"/>
-<junction x="12.7" y="-33.02"/>
+<wire x1="12.7" y1="-30.48" x2="5.08" y2="-30.48" width="0.1524" layer="91"/>
 <pinref part="C3" gate="G$1" pin="2"/>
-<wire x1="-15.24" y1="-27.94" x2="-15.24" y2="-33.02" width="0.1524" layer="91" style="shortdash"/>
+<wire x1="5.08" y1="-30.48" x2="-15.24" y2="-30.48" width="0.1524" layer="91"/>
+<wire x1="-15.24" y1="-30.48" x2="-15.24" y2="-27.94" width="0.1524" layer="91"/>
 <pinref part="C2" gate="G$1" pin="2"/>
-<wire x1="5.08" y1="-27.94" x2="5.08" y2="-33.02" width="0.1524" layer="91" style="shortdash"/>
+<wire x1="5.08" y1="-30.48" x2="5.08" y2="-27.94" width="0.1524" layer="91"/>
+</segment>
+<segment>
+<pinref part="SUPPLY33" gate="GND" pin="GND"/>
+<wire x1="-48.26" y1="5.08" x2="-55.88" y2="5.08" width="0.1524" layer="91"/>
+<pinref part="C5" gate="G$1" pin="2"/>
+<wire x1="-55.88" y1="5.08" x2="-76.2" y2="5.08" width="0.1524" layer="91"/>
+<wire x1="-76.2" y1="5.08" x2="-76.2" y2="7.62" width="0.1524" layer="91"/>
+<pinref part="C4" gate="G$1" pin="2"/>
+<wire x1="-55.88" y1="5.08" x2="-55.88" y2="7.62" width="0.1524" layer="91"/>
 </segment>
 </net>
@@
 <wire x1="-2.54" y1="2.54" x2="-22.86" y2="2.54" width="0.1524" layer="91"/>
 <wire x1="-22.86" y1="2.54" x2="-22.86" y2="-17.78" width="0.1524" layer="91"/>
-<wire x1="-22.86" y1="-17.78" x2="-20.32" y2="-17.78" width="0.1524" layer="91"/>
+<wire x1="-22.86" y1="-17.78" x2="-15.24" y2="-17.78" width="0.1524" layer="91"/>
+<pinref part="C3" gate="G$1" pin="1"/>
+<wire x1="-15.24" y1="-17.78" x2="-10.16" y2="-17.78" width="0.1524" layer="91"/>
+<wire x1="-15.24" y1="-17.78" x2="-15.24" y2="-20.32" width="0.1524" layer="91"/>
 </segment>
 </net>
@@
 </segment>
 </net>
-<net name="N$19" class="0">
-<segment>
-<pinref part="L1" gate="1" pin="1"/>
-<wire x1="-17.78" y1="-17.78" x2="-15.24" y2="-17.78" width="0.1524" layer="91" style="shortdash"/>
-<wire x1="-12.7" y1="-17.78" x2="-15.24" y2="-17.78" width="0.1524" layer="91" style="shortdash"/>
-<pinref part="C3" gate="G$1" pin="1"/>
-<wire x1="-15.24" y1="-17.78" x2="-15.24" y2="-20.32" width="0.1524" layer="91" style="shortdash"/>
-</segment>
-</net>
 <net name="N$20" class="0">
 <segment>
 <pinref part="L1" gate="1" pin="2"/>
 <wire x1="2.54" y1="-17.78" x2="5.08" y2="-17.78" width="0.1524" layer="91" style="shortdash"/>
-<wire x1="12.7" y1="-17.78" x2="5.08" y2="-17.78" width="0.1524" layer="91" style="shortdash"/>
+<wire x1="2.54" y1="-17.78" x2="5.08" y2="-17.78" width="0.1524" layer="91"/>
 <pinref part="C2" gate="G$1" pin="1"/>
-<wire x1="5.08" y1="-17.78" x2="5.08" y2="-20.32" width="0.1524" layer="91" style="shortdash"/>
-</segment>
-</net>
+<wire x1="5.08" y1="-17.78" x2="5.08" y2="-20.32" width="0.1524" layer="91"/>
+<wire x1="5.08" y1="-17.78" x2="20.32" y2="-17.78" width="0.1524" layer="91"/>
+</segment>
+</net>
+<net name="N$34" class="0">
+<segment>
+<pinref part="L2" gate="1" pin="2"/>
+<wire x1="-58.42" y1="17.78" x2="-55.88" y2="17.78" width="0.1524" layer="91" style="shortdash"/>
+<wire x1="-58.42" y1="17.78" x2="-55.88" y2="17.78" width="0.1524" layer="91"/>
+<pinref part="C4" gate="G$1" pin="1"/>
+<wire x1="-55.88" y1="17.78" x2="-55.88" y2="15.24" width="0.1524" layer="91"/>
+<wire x1="-55.88" y1="17.78" x2="-40.64" y2="17.78" width="0.1524" layer="91"/>
+</segment>
+</net>
+<net name="N$35" class="0">
+<segment>
+<wire x1="-83.82" y1="17.78" x2="-76.2" y2="17.78" width="0.1524" layer="91"/>
+<pinref part="C5" gate="G$1" pin="1"/>
+<wire x1="-76.2" y1="17.78" x2="-73.66" y2="17.78" width="0.1524" layer="91"/>
+<wire x1="-73.66" y1="17.78" x2="-71.12" y2="17.78" width="0.1524" layer="91"/>
+<wire x1="-76.2" y1="17.78" x2="-76.2" y2="15.24" width="0.1524" layer="91"/>
+<pinref part="L2" gate="1" pin="1"/>
+<wire x1="-83.82" y1="17.78" x2="-83.82" y2="40.64" width="0.1524" layer="91"/>
+<wire x1="-83.82" y1="40.64" x2="-48.26" y2="40.64" width="0.1524" layer="91"/>
+</segment>
+</net>
+<net name="N$19" class="0">
+<segment>
+<pinref part="J4" gate="-1" pin="MSV"/>
+<wire x1="76.2" y1="-25.4" x2="63.5" y2="-25.4" width="0.1524" layer="91"/>
+</segment>
+</net>
