File: eagle/joesTriac/joesTriac-2nd/cpuConnectionBoard.sch (EAGLE design)
At the start: 24 parts, among them IC1 24C01CP, IC2 LM311N, J1 CN11, J2 CN9, J3 CN13, J4 CN14, J5 CN9, Q1 2N4403, Q2 2N4401

Commit message: candidate for release
Connections:
- net GND: now also J5-6.MS
Other:
- note added: "connector to triac board"
- note added: "gnd needed if cpu and triac boards protected by emi filters"
- note removed: "connector to boards"
Changed lines of the file:
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@@
 <text x="-15.24" y="48.26" size="1.778" layer="91">PH6</text>
 <text x="124.46" y="46.482" size="1.778" layer="91">triac trigger</text>
-<text x="162.56" y="60.96" size="1.778" layer="91">connector to boards</text>
+<text x="162.56" y="60.96" size="1.778" layer="91">connector to triac board</text>
 <text x="139.7" y="31.242" size="1.778" layer="91">VoltageZeroPass</text>
 <text x="-22.86" y="3.302" size="1.778" layer="91">VoltageZeroPass</text>
@@
 <text x="-50.8" y="19.05" size="1.778" layer="91">adc</text>
 <text x="66.04" y="-22.86" size="1.778" layer="91">adc</text>
+<text x="134.62" y="20.32" size="1.778" layer="91">gnd needed if cpu and triac boards protected by emi filters</text>
 </plain>
 <instances>
@@
 <pinref part="R4" gate="G$1" pin="1"/>
 <wire x1="116.84" y1="22.86" x2="116.84" y2="17.78" width="0.1524" layer="91"/>
+<wire x1="116.84" y1="17.78" x2="129.54" y2="17.78" width="0.1524" layer="91"/>
+<wire x1="129.54" y1="17.78" x2="129.54" y2="43.18" width="0.1524" layer="91"/>
+<pinref part="J5" gate="-6" pin="MS"/>
+<wire x1="129.54" y1="43.18" x2="160.02" y2="43.18" width="0.1524" layer="91"/>
 </segment>
 <segment>
