File: eagle/joesTriac/joesTriac-2nd/powerBoard-2nd.sch (EAGLE design)
At the start: 47 parts, among them IC1 7809, IC2 7805, IC3 7909, IC5 7809, IC7 LM311N, IC8 TLC251P, J1 XF2E-0815-1, J2 XF2E-0815-1, J3 XF2E-0815-1, J4 XF2E-0815-1

Commit message: reg save, working on exti
Parts:
- added R12: 2.2k, resistor:R-EU_0309/V
Connections:
- net GND: now also R12.1
- net N$22: now also R12.2
Changed lines of the file:
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@@
 <part name="R17" library="resistor" deviceset="R-EU_" device="0309/V" value="2.2k"/>
 <part name="J4" library="con-omron" deviceset="XF2*-08?" device="15-1" technology="E" value=""/>
+<part name="R12" library="resistor" deviceset="R-EU_" device="0309/V" value="2.2k"/>
 </parts>
 <sheets>
@@
 <instance part="J4" gate="-2" x="48.26" y="68.58" rot="R180"/>
 <instance part="J4" gate="-3" x="48.26" y="71.12" rot="R180"/>
+<instance part="R12" gate="G$1" x="-5.08" y="48.26" rot="R90"/>
 </instances>
 <busses>
@@
 <pinref part="D3" gate="1" pin="A"/>
 <wire x1="0" y1="33.02" x2="0" y2="30.48" width="0.1524" layer="91"/>
+<pinref part="R12" gate="G$1" pin="1"/>
+<wire x1="-5.08" y1="43.18" x2="-5.08" y2="30.48" width="0.1524" layer="91" style="shortdash"/>
+<wire x1="-5.08" y1="30.48" x2="0" y2="30.48" width="0.1524" layer="91" style="shortdash"/>
 </segment>
 <segment>
@@
 <wire x1="-27.94" y1="55.88" x2="-22.86" y2="55.88" width="0.1524" layer="91"/>
 <wire x1="-22.86" y1="55.88" x2="-20.32" y2="55.88" width="0.1524" layer="91"/>
-<wire x1="-20.32" y1="55.88" x2="-12.7" y2="55.88" width="0.1524" layer="91"/>
-<wire x1="-12.7" y1="55.88" x2="-12.7" y2="-15.24" width="0.1524" layer="91"/>
-<wire x1="-12.7" y1="-15.24" x2="-149.86" y2="-15.24" width="0.1524" layer="91"/>
+<wire x1="-20.32" y1="55.88" x2="-15.24" y2="55.88" width="0.1524" layer="91"/>
+<wire x1="-15.24" y1="55.88" x2="-15.24" y2="-15.24" width="0.1524" layer="91"/>
+<wire x1="-15.24" y1="-15.24" x2="-149.86" y2="-15.24" width="0.1524" layer="91"/>
 <wire x1="-149.86" y1="-15.24" x2="-149.86" y2="48.26" width="0.1524" layer="91"/>
 <pinref part="J2" gate="-4" pin="MS"/>
@@
 <segment>
 <wire x1="5.08" y1="71.12" x2="0" y2="71.12" width="0.1524" layer="91"/>
-<wire x1="0" y1="71.12" x2="0" y2="38.1" width="0.1524" layer="91"/>
+<wire x1="0" y1="71.12" x2="0" y2="66.04" width="0.1524" layer="91"/>
 <pinref part="D3" gate="1" pin="C"/>
 <pinref part="R14" gate="G$1" pin="2"/>
+<wire x1="0" y1="66.04" x2="0" y2="38.1" width="0.1524" layer="91"/>
 <wire x1="5.08" y1="40.64" x2="10.16" y2="40.64" width="0.1524" layer="91"/>
 <wire x1="5.08" y1="71.12" x2="5.08" y2="43.18" width="0.1524" layer="91"/>
@@
 <wire x1="7.62" y1="73.66" x2="5.08" y2="73.66" width="0.1524" layer="91"/>
 <wire x1="5.08" y1="73.66" x2="5.08" y2="71.12" width="0.1524" layer="91"/>
-</segment>
-</net>
+<wire x1="0" y1="66.04" x2="-5.08" y2="66.04" width="0.1524" layer="91" style="shortdash"/>
+<wire x1="-5.08" y1="66.04" x2="-5.08" y2="53.34" width="0.1524" layer="91" style="shortdash"/>
+<pinref part="R12" gate="G$1" pin="2"/>
+</segment>
+</net>

Commit message: candidate for release
Other:
- note added: "zero pass signal, not implemented"
- note removed: "zero pass signal"
Changed lines of the file:
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@@
 <text x="-124.46" y="60.96" size="1.778" layer="91">/+16V</text>
 <text x="-127" y="-10.16" size="1.778" layer="91">/-16V</text>
-<text x="49.276" y="21.59" size="1.9304" layer="91">zero pass signal</text>
+<text x="26.416" y="21.59" size="1.9304" layer="91">zero pass signal, not implemented</text>
 <text x="22.86" y="65.278" size="1.778" layer="91">hysterese</text>
+<wire x1="-5.08" y1="101.6" x2="-5.08" y2="91.44" width="0.1524" layer="99"/>
+<wire x1="-5.08" y1="91.44" x2="2.54" y2="91.44" width="0.1524" layer="99"/>
+<wire x1="2.54" y1="91.44" x2="2.54" y2="73.66" width="0.1524" layer="99"/>
+<wire x1="2.54" y1="73.66" x2="-2.54" y2="73.66" width="0.1524" layer="99"/>
+<wire x1="-2.54" y1="73.66" x2="-2.54" y2="68.58" width="0.1524" layer="99"/>
+<wire x1="-2.54" y1="68.58" x2="-5.08" y2="66.04" width="0.1524" layer="99"/>
+<wire x1="-5.08" y1="66.04" x2="-10.16" y2="66.04" width="0.1524" layer="99"/>
+<wire x1="-10.16" y1="66.04" x2="-10.16" y2="22.86" width="0.1524" layer="99"/>
+<wire x1="-10.16" y1="22.86" x2="20.32" y2="22.86" width="0.1524" layer="99"/>
+<wire x1="20.32" y1="22.86" x2="20.32" y2="20.32" width="0.1524" layer="99"/>
+<wire x1="20.32" y1="20.32" x2="73.66" y2="20.32" width="0.1524" layer="99"/>
+<wire x1="73.66" y1="20.32" x2="73.66" y2="101.6" width="0.1524" layer="99"/>
+<wire x1="73.66" y1="101.6" x2="-5.08" y2="101.6" width="0.1524" layer="99"/>
 </plain>
 <instances>
