File: eagle/joesTriac/joesTriac-2nd/triacBoard.sch (EAGLE design)
At the start: 13 parts, among them X1 1751316, X2 1751248

Commit message: reg save, working on exti spikes
Parts:
- added C4: 47nF, resistor:C-EU050-030X075
- added C5: 22nF, resistor:C-EU050-030X075
- added L2: SMCC12, inductors:SMCC12
Connections:
- removed net N$15: OK1A.C, R8.1, X2-2.K
- new net N$3: OK1A.C, R8.1
- new net N$34: C4.1, L2.2, X2-2.K
- new net N$35: C5.1, L2.1
- net GND: now also C4.2, C5.2
Changed lines of the file:
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@@
 <layer number="51" name="tDocu" color="7" fill="1" visible="no" active="no"/>
 <layer number="52" name="bDocu" color="7" fill="1" visible="no" active="no"/>
+<layer number="90" name="Modules" color="5" fill="1" visible="yes" active="yes"/>
 <layer number="91" name="Nets" color="2" fill="1" visible="yes" active="yes"/>
 <layer number="92" name="Busses" color="1" fill="1" visible="yes" active="yes"/>
@@
 <layer number="98" name="Guide" color="6" fill="1" visible="yes" active="yes"/>
 <layer number="99" name="SpiceOrder" color="5" fill="1" visible="yes" active="yes"/>
+<layer number="101" name="Hidden" color="15" fill="1" visible="yes" active="yes"/>
+<layer number="102" name="Changes" color="12" fill="1" visible="yes" active="yes"/>
 </layers>
 <schematic xreflabel="%F%N/%S.%C%R" xrefpart="/%S.%C%R">
@@
 <part name="SUPPLY1" library="supply2" deviceset="GND" device=""/>
 <part name="C2" library="resistor" deviceset="C-EU" device="025-040X050" value="0.05U"/>
+<part name="L2" library="inductors" deviceset="SMCC12" device=""/>
+<part name="C4" library="resistor" deviceset="C-EU" device="050-030X075" value="47nF"/>
+<part name="C5" library="resistor" deviceset="C-EU" device="050-030X075" value="22nF"/>
+<part name="SUPPLY33" library="supply2" deviceset="GND" device=""/>
 </parts>
 <sheets>
@@
 <instance part="SUPPLY1" gate="GND" x="-99.06" y="55.88"/>
 <instance part="C2" gate="G$1" x="-60.96" y="66.04"/>
+<instance part="L2" gate="1" x="55.88" y="121.92"/>
+<instance part="C4" gate="G$1" x="66.04" y="116.84"/>
+<instance part="C5" gate="G$1" x="45.72" y="116.84"/>
+<instance part="SUPPLY33" gate="GND" x="73.66" y="106.68"/>
 </instances>
 <busses>
@@
 <pinref part="SUPPLY1" gate="GND" pin="GND"/>
 <wire x1="-99.06" y1="66.04" x2="-99.06" y2="58.42" width="0.1524" layer="91"/>
+</segment>
+<segment>
+<pinref part="SUPPLY33" gate="GND" pin="GND"/>
+<wire x1="73.66" y1="109.22" x2="66.04" y2="109.22" width="0.1524" layer="91"/>
+<pinref part="C5" gate="G$1" pin="2"/>
+<wire x1="66.04" y1="109.22" x2="45.72" y2="109.22" width="0.1524" layer="91"/>
+<wire x1="45.72" y1="109.22" x2="45.72" y2="111.76" width="0.1524" layer="91"/>
+<pinref part="C4" gate="G$1" pin="2"/>
+<wire x1="66.04" y1="109.22" x2="66.04" y2="111.76" width="0.1524" layer="91"/>
 </segment>
 </net>
@@
 </segment>
 </net>
-<net name="N$15" class="0">
-<segment>
-<pinref part="OK1" gate="A" pin="C"/>
-<pinref part="R8" gate="G$1" pin="1"/>
-<wire x1="17.78" y1="121.92" x2="25.4" y2="121.92" width="0.1524" layer="91"/>
-<wire x1="25.4" y1="121.92" x2="25.4" y2="116.84" width="0.1524" layer="91"/>
-<wire x1="129.54" y1="116.84" x2="129.54" y2="25.4" width="0.1524" layer="91"/>
-<wire x1="129.54" y1="25.4" x2="43.18" y2="25.4" width="0.1524" layer="91"/>
-<wire x1="43.18" y1="25.4" x2="43.18" y2="35.56" width="0.1524" layer="91"/>
-<pinref part="X2" gate="-2" pin="K"/>
-<wire x1="43.18" y1="35.56" x2="48.26" y2="35.56" width="0.1524" layer="91"/>
-<wire x1="25.4" y1="116.84" x2="129.54" y2="116.84" width="0.1524" layer="91"/>
-</segment>
-</net>
 <net name="N$2" class="0">
 <segment>
@@
 </segment>
 </net>
+<net name="N$34" class="0">
+<segment>
+<pinref part="L2" gate="1" pin="2"/>
+<wire x1="63.5" y1="121.92" x2="66.04" y2="121.92" width="0.1524" layer="91" style="shortdash"/>
+<wire x1="63.5" y1="121.92" x2="66.04" y2="121.92" width="0.1524" layer="91"/>
+<pinref part="C4" gate="G$1" pin="1"/>
+<wire x1="66.04" y1="121.92" x2="66.04" y2="119.38" width="0.1524" layer="91"/>
+<wire x1="66.04" y1="121.92" x2="129.54" y2="121.92" width="0.1524" layer="91"/>
+<wire x1="129.54" y1="121.92" x2="129.54" y2="25.4" width="0.1524" layer="91"/>
+<wire x1="129.54" y1="25.4" x2="43.18" y2="25.4" width="0.1524" layer="91"/>
+<wire x1="43.18" y1="25.4" x2="43.18" y2="35.56" width="0.1524" layer="91"/>
+<pinref part="X2" gate="-2" pin="K"/>
+<wire x1="43.18" y1="35.56" x2="48.26" y2="35.56" width="0.1524" layer="91"/>
+</segment>
+</net>
+<net name="N$35" class="0">
+<segment>
+<wire x1="38.1" y1="121.92" x2="45.72" y2="121.92" width="0.1524" layer="91"/>
+<pinref part="C5" gate="G$1" pin="1"/>
+<wire x1="45.72" y1="121.92" x2="48.26" y2="121.92" width="0.1524" layer="91"/>
+<wire x1="48.26" y1="121.92" x2="50.8" y2="121.92" width="0.1524" layer="91"/>
+<wire x1="45.72" y1="121.92" x2="45.72" y2="119.38" width="0.1524" layer="91"/>
+<pinref part="L2" gate="1" pin="1"/>
+</segment>
+</net>
+<net name="N$3" class="0">
+<segment>
+<pinref part="R8" gate="G$1" pin="1"/>
+<wire x1="25.4" y1="121.92" x2="25.4" y2="116.84" width="0.1524" layer="91"/>
+<pinref part="OK1" gate="A" pin="C"/>
+<wire x1="17.78" y1="121.92" x2="25.4" y2="121.92" width="0.1524" layer="91"/>
+</segment>
+</net>

Commit message: candidate for release
Other:
- note added: "2505/NJ221"
- note added: "XXXXXXX"
Changed lines of the file:
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@@
 <text x="-93.98" y="60.96" size="1.778" layer="91">=====</text>
 <text x="-88.9" y="60.96" size="1.778" layer="91">=====</text>
+<text x="-2.54" y="111.76" size="1.778" layer="92">XXXXXXX</text>
+<text x="-1.778" y="128.016" size="1.778" layer="91">2505/NJ221</text>
 </plain>
 <instances>
